File: DC_load.kicad_pcb (KiCad board)
At the start: 2 copper layers, 100 x 145 mm, 19 parts, among them J2 4 mm terminal, J3 4 mm terminal, J4 4 mm terminal, J5 4 mm terminal, Q3 IRF3205, Q4 IRF3205, Q5 IRF3205, Q6 IRF3205, SW1 RotaryEncoder_Switch, SW2 RotaryEncoder_Switch, U1 STM32F401RCTx

Commit message: New dimensions.
Parts:
- removed D1, D2: 1N4148W, Diode_SMD:D_SOD-123
- added C1: 100p, Capacitor_SMD:C_0603_1608Metric_Pad1.08x0.95mm_HandSolder, F.Cu at (93.6, 117.0)
- added C10: 100n, Capacitor_SMD:C_0603_1608Metric_Pad1.08x0.95mm_HandSolder, F.Cu at (104.8, 111.4)
- added C11: 100n, Capacitor_SMD:C_0603_1608Metric_Pad1.08x0.95mm_HandSolder, F.Cu at (104.6, 117.0)
- added C2: 100p, Capacitor_SMD:C_0603_1608Metric_Pad1.08x0.95mm_HandSolder, F.Cu at (98.8, 97.0)
- added C20: 100p, Capacitor_SMD:C_0603_1608Metric_Pad1.08x0.95mm_HandSolder, F.Cu at (100.4, 118.8)
- added C3: 100p, Capacitor_SMD:C_0603_1608Metric_Pad1.08x0.95mm_HandSolder, F.Cu at (100.4, 93.0)
- added C4: 100p, Capacitor_SMD:C_0603_1608Metric_Pad1.08x0.95mm_HandSolder, F.Cu at (116.0, 115.8)
- added C46: 100n, Capacitor_SMD:C_0603_1608Metric_Pad1.08x0.95mm_HandSolder, F.Cu at (104.4, 101.2)
- added C5: 100p, Capacitor_SMD:C_0603_1608Metric_Pad1.08x0.95mm_HandSolder, F.Cu at (110.0, 120.2)
- added C6: 100p, Capacitor_SMD:C_0603_1608Metric_Pad1.08x0.95mm_HandSolder, F.Cu at (109.6, 94.2)
- added C7: 100p, Capacitor_SMD:C_0603_1608Metric_Pad1.08x0.95mm_HandSolder, F.Cu at (115.6, 96.4)
- added C8: 100n, Capacitor_SMD:C_0603_1608Metric_Pad1.08x0.95mm_HandSolder, F.Cu at (107.6, 108.6)
- added C9: 100n, Capacitor_SMD:C_0603_1608Metric_Pad1.08x0.95mm_HandSolder, F.Cu at (105.0, 98.0)
- added J1: Conn_Coaxial, Connector_Coaxial:BNC_Amphenol_B6252HB-NPP3G-50_Horizontal, B.Cu at (152.5, 175.6)
- added J6: USB_B, Connector_USB:USB_B_OST_USB-B1HSxx_Horizontal, B.Cu at (59.5, 165.0)
- added R1: 100, Resistor_SMD:R_0603_1608Metric_Pad0.98x0.95mm_HandSolder, F.Cu at (97.8, 118.0)
- added R10: 10k, Resistor_SMD:R_0603_1608Metric_Pad0.98x0.95mm_HandSolder, F.Cu at (118.6, 115.0)
- added R11: 10k, Resistor_SMD:R_0603_1608Metric_Pad0.98x0.95mm_HandSolder, F.Cu at (114.2, 115.8)
- added R12: 100, Resistor_SMD:R_0603_1608Metric_Pad0.98x0.95mm_HandSolder, F.Cu at (119.0, 125.0)
- added R13: 100, Resistor_SMD:R_0603_1608Metric_Pad0.98x0.95mm_HandSolder, F.Cu at (118.6, 116.6)
- added R14: 10 mOhm, Resistor_SMD:R_2512_6332Metric_Pad1.40x3.35mm_HandSolder, F.Cu at (130.2, 126.0)
- added R15: 10 mOhm, Resistor_SMD:R_2512_6332Metric_Pad1.40x3.35mm_HandSolder, F.Cu at (124.1, 81.9)
- added R16: 100, Resistor_SMD:R_0603_1608Metric_Pad0.98x0.95mm_HandSolder, F.Cu at (117.6, 96.4)
- added R17: 100, Resistor_SMD:R_0603_1608Metric_Pad0.98x0.95mm_HandSolder, F.Cu at (124.6, 94.4)
- added R18: 10k, Resistor_SMD:R_0603_1608Metric_Pad0.98x0.95mm_HandSolder, F.Cu at (113.8, 96.4)
- added R19: 10k, Resistor_SMD:R_0603_1608Metric_Pad0.98x0.95mm_HandSolder, F.Cu at (111.4, 96.4)
- added R2: 100, Resistor_SMD:R_0603_1608Metric_Pad0.98x0.95mm_HandSolder, F.Cu at (87.8, 121.2)
- added R3: 10 mOhm, Resistor_SMD:R_2512_6332Metric_Pad1.40x3.35mm_HandSolder, F.Cu at (85.2, 131.2)
- added R31: 10k, Resistor_SMD:R_0603_1608Metric_Pad0.98x0.95mm_HandSolder, F.Cu at (95.2, 117.0)
- added R4: 10k, Resistor_SMD:R_0603_1608Metric_Pad0.98x0.95mm_HandSolder, F.Cu at (90.4, 116.8)
- added R5: 10k, Resistor_SMD:R_0603_1608Metric_Pad0.98x0.95mm_HandSolder, F.Cu at (98.8, 93.6)
- added R6: 10k, Resistor_SMD:R_0603_1608Metric_Pad0.98x0.95mm_HandSolder, F.Cu at (101.2, 98.8)
- added R7: 100, Resistor_SMD:R_0603_1608Metric_Pad0.98x0.95mm_HandSolder, F.Cu at (90.6, 85.8)
- added R8: 100, Resistor_SMD:R_0603_1608Metric_Pad0.98x0.95mm_HandSolder, F.Cu at (97.0, 97.0)
- added R9: 10 mOhm, Resistor_SMD:R_2512_6332Metric_Pad1.40x3.35mm_HandSolder, F.Cu at (80.5, 87.8)
- added U3: NCS21802, Package_SO:OnSemi_Micro8, F.Cu at (104.6, 114.0)
- added U4: NCS21802, Package_SO:OnSemi_Micro8, F.Cu at (105.0, 104.0)
- added U5: TLV9062, Package_SO:SOIC-8_3.9x4.9mm_P1.27mm, F.Cu at (105.0, 120.0)
- added U6: TLV9062, Package_SO:SOIC-8_3.9x4.9mm_P1.27mm, F.Cu at (105.0, 94.2)
- added U7: LMT84LPM, Package_TO_SOT_THT:TO-92_Inline_W4.0mm_Horizontal_FlatSideUp, B.Cu at (109.5, 107.1)
- added U9: CH340C, Package_SO:SOIC-16_3.9x9.9mm_P1.27mm, B.Cu at (56.7, 175.3)
- Q3, Q4, Q5, Q6: value IRF3205 -> FQP19N20C
- U2: value ~ -> Screen
- moved SW2 52.0 mm to (130.0, 185.0), turned to 90 degrees
- moved SW1 45.0 mm to (80.0, 185.0), turned to 90 degrees
- moved J2 10.9 mm to (140.0, 59.0)
- moved J3 10.9 mm to (124.9, 59.0)
- moved H2 10.0 mm to (155.0, 190.0)
- moved H4 10.0 mm to (155.0, 55.0)
- moved U2 5.19 mm to (73.0, 145.9)
- moved HS1 5.00 mm to (105.0, 107.0)
- moved Q3 5.00 mm to (85.1, 123.3)
- moved Q4 5.00 mm to (88.7, 87.1)
- moved Q5 5.00 mm to (121.3, 126.9)
- moved Q6 5.00 mm to (124.9, 90.7)
- moved U1 4.82 mm to (104.8, 187.4)
- moved J4 1.00 mm to (85.1, 59.0)
- moved J5 1.00 mm to (70.0, 59.0)
Connections:
- Q3 pad 1: unconnected-(Q3-G-Pad1) -> Net-(Q3-G)
- Q3 pad 2: unconnected-(Q3-D-Pad2) -> INPUT_POWER
- Q3 pad 3: unconnected-(Q3-S-Pad3) -> Net-(Q3-S)
- Q4 pad 1: unconnected-(Q4-G-Pad1) -> Net-(Q4-G)
- Q4 pad 2: unconnected-(Q4-D-Pad2) -> INPUT_POWER
- Q4 pad 3: unconnected-(Q4-S-Pad3) -> Net-(Q4-S)
- Q5 pad 1: unconnected-(Q5-G-Pad1) -> Net-(Q5-G)
- Q5 pad 2: unconnected-(Q5-D-Pad2) -> INPUT_POWER
- Q5 pad 3: unconnected-(Q5-S-Pad3) -> Net-(Q5-S)
- Q6 pad 1: unconnected-(Q6-G-Pad1) -> Net-(Q6-G)
- Q6 pad 2: unconnected-(Q6-D-Pad2) -> INPUT_POWER
- Q6 pad 3: unconnected-(Q6-S-Pad3) -> Net-(Q6-S)
Routing:
- added copper zone on B.Cu, net GND
- added copper zone on F.Cu, net INPUT_POWER
Other:
- board size 100 x 145 mm -> 110 x 145 mm

Commit message: Schematic progress.
Parts:
- added C12: 1u, Capacitor_SMD:C_2220_5750Metric_Pad1.97x5.40mm_HandSolder, F.Cu at (130.1, 83.7)
- added C13: 1u, Capacitor_SMD:C_2220_5750Metric_Pad1.97x5.40mm_HandSolder, F.Cu at (81.4, 81.8)
- added C14: 1u, Capacitor_SMD:C_2220_5750Metric_Pad1.97x5.40mm_HandSolder, F.Cu at (80.5, 129.6)
- added C15: 1u, Capacitor_SMD:C_2220_5750Metric_Pad1.97x5.40mm_HandSolder, F.Cu at (128.5, 132.3)
- added C16: 100n, Capacitor_SMD:C_0603_1608Metric_Pad1.08x0.95mm_HandSolder, F.Cu at (91.3, 207.7)
- added C17: 100n, Capacitor_SMD:C_0603_1608Metric_Pad1.08x0.95mm_HandSolder, F.Cu at (91.3, 210.2)
- added C18: 100n, Capacitor_SMD:C_0603_1608Metric_Pad1.08x0.95mm_HandSolder, F.Cu at (91.3, 212.7)
- added C19: 100n, Capacitor_SMD:C_0603_1608Metric_Pad1.08x0.95mm_HandSolder, F.Cu at (91.3, 215.2)
- added C21: 10n, Capacitor_SMD:C_0603_1608Metric_Pad1.08x0.95mm_HandSolder, F.Cu at (91.3, 217.7)
- added C22: 100p, Capacitor_SMD:C_0603_1608Metric_Pad1.08x0.95mm_HandSolder, F.Cu at (95.7, 207.7)
- added C23: 10n, Capacitor_SMD:C_0603_1608Metric_Pad1.08x0.95mm_HandSolder, F.Cu at (95.7, 210.2)
- added C24: 100p, Capacitor_SMD:C_0603_1608Metric_Pad1.08x0.95mm_HandSolder, F.Cu at (95.7, 212.7)
- added C25: 10n, Capacitor_SMD:C_0603_1608Metric_Pad1.08x0.95mm_HandSolder, F.Cu at (95.7, 215.2)
- added C26: 100p, Capacitor_SMD:C_0603_1608Metric_Pad1.08x0.95mm_HandSolder, F.Cu at (95.7, 217.7)
- added C27: 10n, Capacitor_SMD:C_0603_1608Metric_Pad1.08x0.95mm_HandSolder, F.Cu at (100.0, 207.7)
- added C28: 100p, Capacitor_SMD:C_0603_1608Metric_Pad1.08x0.95mm_HandSolder, F.Cu at (100.0, 210.2)
- added C29: 100n, Capacitor_SMD:C_0603_1608Metric_Pad1.08x0.95mm_HandSolder, F.Cu at (130.2, 211.3)
- added C30: 10u, Capacitor_SMD:C_0603_1608Metric_Pad1.08x0.95mm_HandSolder, F.Cu at (118.3, 219.6)
- added C31: 10u, Capacitor_SMD:C_0603_1608Metric_Pad1.08x0.95mm_HandSolder, F.Cu at (118.3, 222.1)
- added C32: 100n, Capacitor_SMD:C_0603_1608Metric_Pad1.08x0.95mm_HandSolder, F.Cu at (118.6, 223.6)
- added C33: 100n, Capacitor_SMD:C_0603_1608Metric_Pad1.08x0.95mm_HandSolder, F.Cu at (118.6, 226.1)
- added C34: 10u, Capacitor_SMD:C_0603_1608Metric_Pad1.08x0.95mm_HandSolder, F.Cu at (118.6, 228.6)
- added D1: 1N4148W, Diode_SMD:D_SOD-123, F.Cu at (86.2, 225.8)
- added D2: 1N4148W, Diode_SMD:D_SOD-123, F.Cu at (86.2, 229.1)
- added R20: 100, Resistor_SMD:R_0603_1608Metric_Pad0.98x0.95mm_HandSolder, F.Cu at (85.5, 232.1)
- added R21: 10k, Resistor_SMD:R_0603_1608Metric_Pad0.98x0.95mm_HandSolder, F.Cu at (100.0, 212.7)
- added R22: 100, Resistor_SMD:R_0603_1608Metric_Pad0.98x0.95mm_HandSolder, F.Cu at (100.0, 215.2)
- added R23: 100, Resistor_SMD:R_0603_1608Metric_Pad0.98x0.95mm_HandSolder, F.Cu at (100.0, 217.7)
- added R24: 10k, Resistor_SMD:R_0603_1608Metric_Pad0.98x0.95mm_HandSolder, F.Cu at (104.4, 207.7)
- added R25: 100, Resistor_SMD:R_0603_1608Metric_Pad0.98x0.95mm_HandSolder, F.Cu at (104.4, 210.2)
- added R26: 10k, Resistor_SMD:R_0603_1608Metric_Pad0.98x0.95mm_HandSolder, F.Cu at (104.4, 212.7)
- added R27: 100, Resistor_SMD:R_0603_1608Metric_Pad0.98x0.95mm_HandSolder, F.Cu at (104.4, 215.2)
- added R28: 10k, Resistor_SMD:R_0603_1608Metric_Pad0.98x0.95mm_HandSolder, F.Cu at (104.4, 217.7)
- added R29: 1Meg, Resistor_SMD:R_0603_1608Metric_Pad0.98x0.95mm_HandSolder, F.Cu at (125.5, 223.6)
- added R30: 50k, Resistor_SMD:R_0603_1608Metric_Pad0.98x0.95mm_HandSolder, F.Cu at (125.5, 226.1)
- added R32: 1Meg, Resistor_SMD:R_0603_1608Metric_Pad0.98x0.95mm_HandSolder, F.Cu at (125.5, 228.6)
- added R33: 50k, Resistor_SMD:R_0603_1608Metric_Pad0.98x0.95mm_HandSolder, F.Cu at (125.5, 231.1)
- added R34: 100, Resistor_SMD:R_0603_1608Metric_Pad0.98x0.95mm_HandSolder, F.Cu at (118.6, 231.1)
- added U10: FSA3157P6X, Package_TO_SOT_SMD:SOT-363_SC-70-6_Handsoldering, F.Cu at (86.2, 212.3)
- added U11: FSA3157P6X, Package_TO_SOT_SMD:SOT-363_SC-70-6_Handsoldering, F.Cu at (86.2, 216.3)
- added U12: FSA3157P6X, Package_TO_SOT_SMD:SOT-363_SC-70-6_Handsoldering, F.Cu at (86.2, 220.2)
- added U14: AMS1117-3.3, Package_TO_SOT_SMD:SOT-223-3_TabPin2, F.Cu at (121.0, 214.2)
- added U15: 74HC14D653, Package_SO:SOIC-14_3.9x8.7mm_P1.27mm, F.Cu at (112.2, 227.6)
- added U16: LM4040DBZ-3, Package_TO_SOT_SMD:SOT-23, F.Cu at (118.9, 234.8)
- added U8: STM32F103C8Tx, Package_QFP:LQFP-48_7x7mm_P0.5mm, B.Cu at (102.9, 186.4)
- J2: value 4 mm terminal -> red_terminal
- J5: value 4 mm terminal -> black terminal
- U1: value STM32F401RCTx -> FSA3157P6X; footprint Package_QFP:LQFP-64_10x10mm_P0.5mm -> Package_TO_SOT_SMD:SOT-363_SC-70-6_Handsoldering; moved to F.Cu
- moved U1 28.0 mm to (86.2, 208.4)
- moved C8 3.62 mm to (110.8, 106.9)
- moved R3 1.64 mm to (86.5, 132.2)
- moved U7 1.46 mm to (109.1, 105.7)
- moved R9 1.03 mm to (79.6, 88.3)
- moved R15 0.42 mm to (123.8, 81.6)
- moved R14 0.30 mm to (130.5, 126.0)
Connections:
- C46 pad 2: 5V -> 3V3
- C9 pad 2: 5V -> 3V3
- J1 pad 1: BNC_CONTROL -> Net-(J1-In)
- J2 pad 1: unconnected-(J2-Pin_1-Pad1) -> V_SENSE+
- J5 pad 1: unconnected-(J5-Pin_1-Pad1) -> V_SENSE-
- U1 pad 1: unconnected-(U1-VBAT-Pad1) -> BNC_CONTROL
- U1 pad 2: unconnected-(U1-PC13-Pad2) -> GND
- U1 pad 3: unconnected-(U1-PC14-Pad3) -> CH1_MCU_CONTROL
- U1 pad 4: unconnected-(U1-PC15-Pad4) -> CH1_CONTROL
- U1 pad 5: unconnected-(U1-PH0-Pad5) -> 5V
- U1 pad 6: unconnected-(U1-PH1-Pad6) -> CH1_SEL
- U3 pad 8: 5V -> 3V3
- U4 pad 8: 5V -> 3V3
