File: kicad/DC_load_front_plate/DC_load_front_plate.kicad_pcb (KiCad board)
At the start: 2 copper layers, 110 x 55 mm, 4 parts

Commit message: aethetics.
Parts:
- moved H3 10.0 mm to (55.0, 135.0)
- moved H4 10.0 mm to (155.0, 135.0)
Routing:
- added copper zone on F.Cu, net 3V3
Other:
- board size 110 x 55 mm -> 110 x 65 mm
- board text added: "DC load"
