File: kicad/DC_load_isolation_module/DC_load_isolation_module.kicad_pcb (KiCad board)
At the start: 2 copper layers, 110 x 145 mm, 32 parts, among them J6 USB_B, Q1 MMBT5401, U14 AMS1117-3.3, U17 CH340C, U18 TL431DBZ, U3 LTV-817S

Commit message: Schematic done.
Parts:
- removed R50: 100, Resistor_SMD:R_0603_1608Metric_Pad0.98x0.95mm_HandSolder
- added C1: 100n, Capacitor_SMD:C_0603_1608Metric_Pad1.08x0.95mm_HandSolder, F.Cu at (199.3, 134.4)
- added C10: 10u, Capacitor_SMD:C_0603_1608Metric_Pad1.08x0.95mm_HandSolder, F.Cu at (165.2, 136.9)
- added C11: 10u, Capacitor_SMD:C_0603_1608Metric_Pad1.08x0.95mm_HandSolder, F.Cu at (165.2, 139.4)
- added C12: 10u, Capacitor_SMD:C_0603_1608Metric_Pad1.08x0.95mm_HandSolder, F.Cu at (165.2, 142.0)
- added C13: 100p, Capacitor_SMD:C_0603_1608Metric_Pad1.08x0.95mm_HandSolder, F.Cu at (165.2, 144.5)
- added C14: 100n, Capacitor_SMD:C_0603_1608Metric_Pad1.08x0.95mm_HandSolder, F.Cu at (165.2, 147.0)
- added C15: 10u, Capacitor_SMD:C_0603_1608Metric_Pad1.08x0.95mm_HandSolder, F.Cu at (165.2, 149.5)
- added C16: 10u, Capacitor_SMD:C_0603_1608Metric_Pad1.08x0.95mm_HandSolder, F.Cu at (165.2, 152.0)
- added C17: 10u, Capacitor_SMD:C_0603_1608Metric_Pad1.08x0.95mm_HandSolder, F.Cu at (165.2, 154.5)
- added C18: 10u, Capacitor_SMD:C_0603_1608Metric_Pad1.08x0.95mm_HandSolder, F.Cu at (169.6, 134.4)
- added C19: 10u, Capacitor_SMD:C_0603_1608Metric_Pad1.08x0.95mm_HandSolder, F.Cu at (169.6, 136.9)
- added C2: 220p, Capacitor_SMD:C_0603_1608Metric_Pad1.08x0.95mm_HandSolder, F.Cu at (199.3, 165.4)
- added C20: 10u, Capacitor_SMD:C_0603_1608Metric_Pad1.08x0.95mm_HandSolder, F.Cu at (169.6, 139.4)
- added C21: 10u, Capacitor_SMD:C_0603_1608Metric_Pad1.08x0.95mm_HandSolder, F.Cu at (169.6, 142.0)
- added C22: 10u, Capacitor_SMD:C_0603_1608Metric_Pad1.08x0.95mm_HandSolder, F.Cu at (169.6, 144.5)
- added C23: 100n, Capacitor_SMD:C_0603_1608Metric_Pad1.08x0.95mm_HandSolder, F.Cu at (169.6, 147.0)
- added C24: 10u, Capacitor_SMD:C_0603_1608Metric_Pad1.08x0.95mm_HandSolder, F.Cu at (169.6, 149.5)
- added C25: 10u, Capacitor_SMD:C_0603_1608Metric_Pad1.08x0.95mm_HandSolder, F.Cu at (169.6, 152.0)
- added C26: 10u, Capacitor_SMD:C_0603_1608Metric_Pad1.08x0.95mm_HandSolder, F.Cu at (169.6, 154.5)
- added C27: 10n, Capacitor_SMD:C_0603_1608Metric_Pad1.08x0.95mm_HandSolder, F.Cu at (199.3, 136.9)
- added C28: 1n, Capacitor_SMD:C_0603_1608Metric_Pad1.08x0.95mm_HandSolder, F.Cu at (199.3, 139.4)
- added C29: 1n, Capacitor_SMD:C_0603_1608Metric_Pad1.08x0.95mm_HandSolder, F.Cu at (199.3, 142.0)
- added C3: 220p, Capacitor_SMD:C_0603_1608Metric_Pad1.08x0.95mm_HandSolder, F.Cu at (199.3, 167.9)
- added C4: 100n, Capacitor_SMD:C_0603_1608Metric_Pad1.08x0.95mm_HandSolder, F.Cu at (199.3, 170.4)
- added C45: 100n, Capacitor_SMD:C_0603_1608Metric_Pad1.08x0.95mm_HandSolder, F.Cu at (173.9, 134.4)
- added C46: 1u, Capacitor_SMD:C_0603_1608Metric_Pad1.08x0.95mm_HandSolder, F.Cu at (173.9, 136.9)
- added C5: 10u, Capacitor_SMD:C_0603_1608Metric_Pad1.08x0.95mm_HandSolder, F.Cu at (199.3, 172.9)
- added C54: 10u, Capacitor_SMD:C_0603_1608Metric_Pad1.08x0.95mm_HandSolder, F.Cu at (203.7, 165.4)
- added C55: 100n, Capacitor_SMD:C_0603_1608Metric_Pad1.08x0.95mm_HandSolder, F.Cu at (203.7, 167.9)
- added C6: 10u, Capacitor_SMD:C_0603_1608Metric_Pad1.08x0.95mm_HandSolder, F.Cu at (199.3, 175.4)
- added C61: 10u, Capacitor_SMD:C_0603_1608Metric_Pad1.08x0.95mm_HandSolder, F.Cu at (203.7, 170.4)
- added C62: 10u, Capacitor_SMD:C_0603_1608Metric_Pad1.08x0.95mm_HandSolder, F.Cu at (203.7, 172.9)
- added C63: 10u, Capacitor_SMD:C_0603_1608Metric_Pad1.08x0.95mm_HandSolder, F.Cu at (203.7, 175.4)
- added C7: 10u, Capacitor_SMD:C_0603_1608Metric_Pad1.08x0.95mm_HandSolder, F.Cu at (199.3, 177.9)
- added C8: 10u, Capacitor_SMD:C_0603_1608Metric_Pad1.08x0.95mm_HandSolder, F.Cu at (199.3, 180.4)
- added C9: 100n, Capacitor_SMD:C_0603_1608Metric_Pad1.08x0.95mm_HandSolder, F.Cu at (165.2, 134.4)
- added D1: BAV99, Package_TO_SOT_SMD:SOT-23, F.Cu at (199.6, 150.6)
- added D11: BAV99, Package_TO_SOT_SMD:SOT-23, F.Cu at (199.6, 159.9)
- added D12: BAV99, Package_TO_SOT_SMD:SOT-23, F.Cu at (204.5, 150.6)
- added D13: BAV99, Package_TO_SOT_SMD:SOT-23, F.Cu at (204.5, 155.3)
- added D14: BAV99, Package_TO_SOT_SMD:SOT-23, F.Cu at (204.5, 159.9)
- added D15: BAV99, Package_TO_SOT_SMD:SOT-23, F.Cu at (182.9, 150.3)
- added D2: BAV99, Package_TO_SOT_SMD:SOT-23, F.Cu at (199.6, 155.3)
- added D3: 1N5819WS, Diode_SMD:D_SOD-323, F.Cu at (182.6, 134.7)
- added D4: 1N5819WS, Diode_SMD:D_SOD-323, F.Cu at (182.6, 137.6)
- added D5: 1N5819WS, Diode_SMD:D_SOD-323, F.Cu at (207.8, 183.2)
- added D7: 1N5819WS, Diode_SMD:D_SOD-323, F.Cu at (182.6, 140.6)
- added D8: 1N5819WS, Diode_SMD:D_SOD-323, F.Cu at (182.6, 143.5)
- added D9: 1N5819WS, Diode_SMD:D_SOD-323, F.Cu at (182.6, 146.4)
- added H3: MountingHole, DC_load:M3_hole_with_spacer, F.Cu at (166.6, 171.7)
- added H4: MountingHole, DC_load:M3_hole_with_spacer, F.Cu at (166.6, 178.7)
- added JP1: Jumper_2_Open, Jumper:SolderJumper-2_P1.3mm_Open_RoundedPad1.0x1.5mm, F.Cu at (217.3, 165.9)
- added JP2: Jumper_2_Open, Jumper:SolderJumper-2_P1.3mm_Open_RoundedPad1.0x1.5mm, F.Cu at (186.9, 134.9)
- added JP3: Jumper_2_Open, Jumper:SolderJumper-2_P1.3mm_Open_RoundedPad1.0x1.5mm, F.Cu at (217.3, 169.4)
- added JP4: Jumper_2_Open, Jumper:SolderJumper-2_P1.3mm_Open_RoundedPad1.0x1.5mm, F.Cu at (186.9, 138.5)
- added JP5: Jumper_2_Open, Jumper:SolderJumper-2_P1.3mm_Open_RoundedPad1.0x1.5mm, F.Cu at (186.9, 142.1)
- added L1: 220u, DC_load:L_Bourns_SRN6045TA, F.Cu at (175.5, 159.5)
- added L4: 220u, DC_load:L_Bourns_SRN6045TA, F.Cu at (214.2, 181.8)
- added Q10: AO3400A, Package_TO_SOT_SMD:SOT-23, F.Cu at (187.8, 150.3)
- added Q11: AO3400A, Package_TO_SOT_SMD:SOT-23, F.Cu at (187.8, 154.9)
- added Q12: MMBT5551L, Package_TO_SOT_SMD:SOT-23, F.Cu at (187.8, 159.6)
- added Q13: AO3400A, Package_TO_SOT_SMD:SOT-23, F.Cu at (212.7, 175.8)
- added Q14: MMBT5401, Package_TO_SOT_SMD:SOT-23, F.Cu at (192.7, 150.3)
- added Q15: MMBT5551L, Package_TO_SOT_SMD:SOT-23, F.Cu at (192.7, 154.9)
- added Q16: MMBT5551L, Package_TO_SOT_SMD:SOT-23, F.Cu at (192.7, 159.6)
- added Q17: MMBT5401, Package_TO_SOT_SMD:SOT-23, F.Cu at (214.4, 155.3)
- added Q18: MMBT5401, Package_TO_SOT_SMD:SOT-23, F.Cu at (214.4, 159.9)
- added Q2: MMBT5401, Package_TO_SOT_SMD:SOT-23, F.Cu at (209.4, 150.6)
- added Q3: MMBT5401, Package_TO_SOT_SMD:SOT-23, F.Cu at (209.4, 155.3)
- added Q4: MMBT5551L, Package_TO_SOT_SMD:SOT-23, F.Cu at (209.4, 159.9)
- added Q5: MMBT5401, Package_TO_SOT_SMD:SOT-23, F.Cu at (212.7, 166.5)
- added Q6: MMBT5551L, Package_TO_SOT_SMD:SOT-23, F.Cu at (212.7, 171.1)
- added Q7: MMBT5551L, Package_TO_SOT_SMD:SOT-23, F.Cu at (214.4, 150.6)
- added Q8: MMBT5551L, Package_TO_SOT_SMD:SOT-23, F.Cu at (182.9, 154.9)
- added Q9: MMBT5401, Package_TO_SOT_SMD:SOT-23, F.Cu at (182.9, 159.6)
- added R1: 1k, Resistor_SMD:R_0603_1608Metric_Pad0.98x0.95mm_HandSolder, F.Cu at (199.3, 144.5)
- added R10: 10, Resistor_SMD:R_0603_1608Metric_Pad0.98x0.95mm_HandSolder, F.Cu at (203.7, 180.4)
- added R11: 100m, Resistor_SMD:R_1206_3216Metric_Pad1.30x1.75mm_HandSolder, F.Cu at (218.1, 172.9)
- added R12: 100m, Resistor_SMD:R_1206_3216Metric_Pad1.30x1.75mm_HandSolder, F.Cu at (218.1, 176.2)
- added R13: 100k, Resistor_SMD:R_0603_1608Metric_Pad0.98x0.95mm_HandSolder, F.Cu at (208.1, 165.4)
- added R14: 1k, Resistor_SMD:R_0603_1608Metric_Pad0.98x0.95mm_HandSolder, F.Cu at (173.9, 139.4)
- added R15: 10, Resistor_SMD:R_0603_1608Metric_Pad0.98x0.95mm_HandSolder, F.Cu at (173.9, 142.0)
- added R16: 100k, Resistor_SMD:R_0603_1608Metric_Pad0.98x0.95mm_HandSolder, F.Cu at (173.9, 144.5)
- added R17: 470k, Resistor_SMD:R_0603_1608Metric_Pad0.98x0.95mm_HandSolder, F.Cu at (173.9, 147.0)
- added R18: 10, Resistor_SMD:R_0603_1608Metric_Pad0.98x0.95mm_HandSolder, F.Cu at (208.1, 134.4)
- added R19: 1k, Resistor_SMD:R_0603_1608Metric_Pad0.98x0.95mm_HandSolder, F.Cu at (173.9, 149.5)
- added R2: 100, Resistor_SMD:R_0603_1608Metric_Pad0.98x0.95mm_HandSolder, F.Cu at (199.3, 147.0)
- added R20: 10, Resistor_SMD:R_0603_1608Metric_Pad0.98x0.95mm_HandSolder, F.Cu at (173.9, 152.0)
- added R21: 100k, Resistor_SMD:R_0603_1608Metric_Pad0.98x0.95mm_HandSolder, F.Cu at (173.9, 154.5)
- added R22: 1k, Resistor_SMD:R_0603_1608Metric_Pad0.98x0.95mm_HandSolder, F.Cu at (178.3, 134.4)
- added R23: 1k, Resistor_SMD:R_0603_1608Metric_Pad0.98x0.95mm_HandSolder, F.Cu at (178.3, 136.9)
- added R24: 39k, Resistor_SMD:R_0603_1608Metric_Pad0.98x0.95mm_HandSolder, F.Cu at (178.3, 139.4)
- added R25: 2.2k, Resistor_SMD:R_0603_1608Metric_Pad0.98x0.95mm_HandSolder, F.Cu at (208.1, 136.9)
- added R26: 10, Resistor_SMD:R_0603_1608Metric_Pad0.98x0.95mm_HandSolder, F.Cu at (208.1, 139.4)
- added R27: 100k, Resistor_SMD:R_0603_1608Metric_Pad0.98x0.95mm_HandSolder, F.Cu at (178.3, 142.0)
- added R28: 10k, Resistor_SMD:R_0603_1608Metric_Pad0.98x0.95mm_HandSolder, F.Cu at (208.1, 142.0)
- added R3: 220, Resistor_SMD:R_0603_1608Metric_Pad0.98x0.95mm_HandSolder, F.Cu at (203.7, 134.4)
- added R37: 100k, Resistor_SMD:R_0603_1608Metric_Pad0.98x0.95mm_HandSolder, F.Cu at (178.3, 144.5)
- added R38: 100k, Resistor_SMD:R_0603_1608Metric_Pad0.98x0.95mm_HandSolder, F.Cu at (208.1, 167.9)
- added R39: 470k, Resistor_SMD:R_0603_1608Metric_Pad0.98x0.95mm_HandSolder, F.Cu at (178.3, 147.0)
- added R4: 100, Resistor_SMD:R_0603_1608Metric_Pad0.98x0.95mm_HandSolder, F.Cu at (203.7, 136.9)
- added R5: 220, Resistor_SMD:R_0603_1608Metric_Pad0.98x0.95mm_HandSolder, F.Cu at (203.7, 139.4)
- added R6: 1k, Resistor_SMD:R_0603_1608Metric_Pad0.98x0.95mm_HandSolder, F.Cu at (203.7, 142.0)
- added R60: 1Meg, Resistor_SMD:R_0603_1608Metric_Pad0.98x0.95mm_HandSolder, F.Cu at (208.1, 170.4)
- added R65: 10k, Resistor_SMD:R_0603_1608Metric_Pad0.98x0.95mm_HandSolder, F.Cu at (208.1, 172.9)
- added R7: 10k, Resistor_SMD:R_0603_1608Metric_Pad0.98x0.95mm_HandSolder, F.Cu at (203.7, 144.5)
- added R8: 10k, Resistor_SMD:R_0603_1608Metric_Pad0.98x0.95mm_HandSolder, F.Cu at (203.7, 147.0)
- added R9: 1k, Resistor_SMD:R_0603_1608Metric_Pad0.98x0.95mm_HandSolder, F.Cu at (203.7, 177.9)
- added U1: LTV-817S, Package_DIP:SMDIP-4_W9.53mm, F.Cu at (216.8, 136.5)
- added U2: MC34063AD, Package_SO:SOIC-8_3.9x4.9mm_P1.27mm, F.Cu at (201.4, 185.0)
- added U5: 74HC14D653, Package_SO:SOIC-14_3.9x8.7mm_P1.27mm, F.Cu at (167.3, 161.0)
- J6: moved to F.Cu
- moved R48 167.5 mm to (217.7, 212.3), turned to 0 degrees
- moved C30 166.7 mm to (209.0, 212.3), turned to 0 degrees
- moved C48 166.1 mm to (213.3, 217.3), turned to 0 degrees
- moved R49 164.8 mm to (217.7, 214.8), turned to 0 degrees
- moved C43 164.7 mm to (213.3, 212.3), turned to 0 degrees
- moved C31 163.3 mm to (209.0, 214.8)
- moved U14 162.9 mm to (191.6, 235.8), turned to 0 degrees
- moved J6 160.6 mm to (196.7, 230.1)
- moved C44 158.7 mm to (213.3, 214.8), turned to 0 degrees
- moved C42 158.3 mm to (209.0, 224.8), turned to 0 degrees
- moved R58 126.7 mm to (217.7, 222.3)
- moved D6 122.7 mm to (209.2, 228.5), turned to 0 degrees
- moved R35 122.1 mm to (213.3, 224.8), turned to 0 degrees
- moved R56 121.6 mm to (217.7, 217.3), turned to 0 degrees
- moved Q1 120.8 mm to (209.2, 233.1)
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Connections:
- C42 pad 2: GND -> Earth
- C43 pad 2: GND -> Earth
- C44 pad 1: GND -> Earth
- C48 pad 1: GND -> Earth
- C57 pad 2: GND -> Earth
- J6 pad 4: GND -> Earth
- J6 pad 5: GND -> Earth
- TP5 pad 1: GND -> Earth
- U17 pad 1: GND -> Earth
- U17 pad 16: 3V3 -> 5V
- U17 pad 2: Net-(U17-TXD) -> TX
- U3 pad 1: unconnected-(U3-Pad1) -> Net-(R3-Pad2)
Routing:
- net (no net): track 2258.4 -> 565.7 mm, vias 56 -> 0
- net GND: track 129.9 -> 37.9 mm, vias 60 -> 0
- net VREF: track 87.0 -> 6.19 mm, vias 2 -> 0
- net TX: track 48.3 -> 4.94 mm, vias 1 -> 0
- net 5V: track 96.6 -> 74.8 mm, vias 20 -> 0
- net 3V3: track 99.6 -> 87.6 mm, vias 29 -> 0
- net Net-(Q7-B): track 103.7 -> 95.8 mm, vias 1 -> 0
- net Net-(D6-A): track 6.45 -> 0.00 mm
- net Net-(J6-D+): track 6.49 -> 1.91 mm, vias 1 -> 0
- net Net-(J6-D-): track 5.61 -> 1.86 mm, vias 1 -> 0
- net Net-(U18-REF): track 3.34 -> 0.00 mm
- net Net-(U17-TXD): track 3.07 -> 0.00 mm, vias 1 -> 0
- net Net-(U17-UD+): track 4.38 -> 1.43 mm, vias 1 -> 0
- net Net-(U17-V3): track 3.60 -> 1.41 mm, vias 1 -> 0
- net Net-(Q1-E): track 1.83 -> 0.00 mm
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- removed copper zone on F.Cu, net (none)
- removed copper zone on F.Cu, net 5V
- removed copper zone on F.Cu, net Net-(Q7-B)

Commit message: kk
Parts:
- added T1: UMEC_UT20A13S, DC_load:UMEC_UT20A13S, F.Cu at (115.8, 170.2)

Commit message: Some placement.
Parts:
- added C32: 100n, Capacitor_SMD:C_0603_1608Metric_Pad1.08x0.95mm_HandSolder, F.Cu at (110.7, 188.7)
- JP2, JP4, JP5: moved to B.Cu
- TP1, TP2, TP3, TP4, TP5, U17: moved to F.Cu
- moved TP5 173.7 mm to (205.2, 55.0)
- moved U17 167.2 mm to (201.5, 89.0)
- moved TP1 164.6 mm to (200.0, 55.0)
- moved U1 159.2 mm to (86.7, 228.3)
- moved C1 142.7 mm to (81.1, 214.4)
- moved C29 142.7 mm to (81.1, 221.9)
- moved D13 142.7 mm to (86.3, 235.2)
- moved D14 142.7 mm to (86.3, 239.8)
- moved D2 142.7 mm to (81.4, 235.2)
- moved Q18 142.7 mm to (96.1, 239.8)
- moved R26 142.7 mm to (89.8, 219.4)
- moved R28 142.7 mm to (89.8, 221.9)
- moved Q3 142.7 mm to (91.2, 235.2)
- moved Q4 142.7 mm to (91.2, 239.8)
- moved R4 142.7 mm to (85.5, 216.9)
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Connections:
- U5 pad 1: GND -> Net-(C13-Pad2)
- U5 pad 12: ~{BF_GATE} -> unconnected-(U5-Pad12)
- U5 pad 13: ~{TF_GATE} -> GND
- U5 pad 2: unconnected-(U5-Pad2) -> ~{TF_GATE}
- U5 pad 3: GND -> ~{TF_GATE}
- U5 pad 4: unconnected-(U5-Pad4) -> ~{BF_GATE}
- U5 pad 8: ~{TF_GATE} -> unconnected-(U5-Pad8)
- U5 pad 9: Net-(C13-Pad2) -> GND
Routing:
- net (no net): track 565.7 -> 0.00 mm
- net Net-(Q7-B): track 95.8 -> 0.00 mm
- net 3V3: track 87.6 -> 0.00 mm
- net 5V: track 74.8 -> 0.00 mm
- net GND: track 37.9 -> 0.00 mm
- net Net-(Q7-E): track 10.1 -> 0.00 mm
- net VREF: track 6.19 -> 0.00 mm
- net TX: track 4.94 -> 0.00 mm
- net Net-(J6-D+): track 1.91 -> 0.00 mm
- net Net-(J6-D-): track 1.86 -> 0.00 mm
- net Net-(U17-UD-): track 1.49 -> 0.00 mm
- net Net-(U17-UD+): track 1.43 -> 0.00 mm
- net Net-(U17-V3): track 1.41 -> 0.00 mm
- net RX: track 1.40 -> 0.00 mm

Commit message: lay.
Parts:
- moved C2 79.3 mm to (131.6, 206.6)
- moved C3 79.3 mm to (131.6, 209.1)
- moved C4 79.3 mm to (131.6, 211.6)
- moved C5 79.3 mm to (131.6, 214.1)
- moved C6 79.3 mm to (131.6, 216.7)
- moved C7 79.3 mm to (131.6, 219.2)
- moved C8 79.3 mm to (131.6, 221.7)
- moved JP1 79.3 mm to (149.5, 207.1)
- moved JP3 79.3 mm to (149.5, 210.7)
- moved L4 79.3 mm to (146.5, 223.0)
- moved Q13 79.3 mm to (144.9, 217.0)
- moved Q5 79.3 mm to (144.9, 207.8)
- moved Q6 79.3 mm to (144.9, 212.4)
- moved R11 79.3 mm to (150.3, 214.1)
- moved R12 79.3 mm to (150.3, 217.4)
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
Commit message: M
Parts:
- removed C35, C57: 10u, Capacitor_SMD:C_0603_1608Metric_Pad1.08x0.95mm_HandSolder
- removed C42, C43: 47p, Capacitor_SMD:C_0603_1608Metric_Pad1.08x0.95mm_HandSolder
- removed C44: 10n, Capacitor_SMD:C_0603_1608Metric_Pad1.08x0.95mm_HandSolder
- removed C48: 100n, Capacitor_SMD:C_0603_1608Metric_Pad1.08x0.95mm_HandSolder
- removed J6: USB_B, DC_load:62910416121
- removed Q1: MMBT5401, Package_TO_SOT_SMD:SOT-23
- removed R48, R49: 22, Resistor_SMD:R_0603_1608Metric_Pad0.98x0.95mm_HandSolder
- removed R56, R58: 10k, Resistor_SMD:R_0603_1608Metric_Pad0.98x0.95mm_HandSolder
- removed R57: 49.9k, Resistor_SMD:R_0603_1608Metric_Pad0.98x0.95mm_HandSolder
- removed TP1, TP4, TP5: TestPoint, TestPoint:TestPoint_Pad_D2.0mm
- removed U14: AMS1117-3.3, Package_TO_SOT_SMD:SOT-223-3_TabPin2
- removed U17: CH340C, Package_SO:SOIC-16_3.9x9.9mm_P1.27mm
- removed U18: TL431DBZ, Package_TO_SOT_SMD:SOT-23
- added D10: GREEN_LED, LED_SMD:LED_0805_2012Metric_Pad1.15x1.40mm_HandSolder, B.Cu at (61.6, 144.1)
- added D16: GREEN_LED, LED_SMD:LED_0805_2012Metric_Pad1.15x1.40mm_HandSolder, B.Cu at (143.7, 182.3)
- added D17: 1N5819WS, Diode_SMD:D_SOD-323, B.Cu at (86.3, 152.2)
- added J12: Iso board connector, Connector_PinSocket_2.54mm:PinSocket_1x08_P2.54mm_Vertical, B.Cu at (151.7, 153.7)
- added J2: USB_C_Receptacle_USB2.0_16P, Connector_USB:USB_C_Receptacle_G-Switch_GT-USB-7010ASV, B.Cu at (70.0, 141.0)
- added R29: 22, Resistor_SMD:R_0603_1608Metric_Pad0.98x0.95mm_HandSolder, B.Cu at (69.0, 153.8)
- added R30: 22, Resistor_SMD:R_0603_1608Metric_Pad0.98x0.95mm_HandSolder, B.Cu at (70.5, 153.8)
- added R31: 10k, Resistor_SMD:R_0603_1608Metric_Pad0.98x0.95mm_HandSolder, B.Cu at (93.2, 151.3)
- added R32: 1k, Resistor_SMD:R_0603_1608Metric_Pad0.98x0.95mm_HandSolder, B.Cu at (61.7, 142.0)
- added R33: 10k, Resistor_SMD:R_0603_1608Metric_Pad0.98x0.95mm_HandSolder, B.Cu at (141.6, 182.7)
- added U4: CH340C, Package_SO:SOIC-16_3.9x9.9mm_P1.27mm, B.Cu at (68.4, 159.5)
- C1, C10, C11, C12, C13, C14, C15, C16, C17, C18, C19, C2, C20, C21, C22, C23, C24, C25, C26, C27, C28, C29, C3, C30, C32, C4, C45, C46, C5, C54, C55, C6, C61, C62, C63, C7, C8, C9, D1, D11, D12, D13, D14, D15, D2, D3, D4, D5, D7, D8, D9, JP1, JP3, L1, L4, Q10, Q11, Q12, Q13, Q14, Q15, Q16, Q17, Q18, Q2, Q3, Q4, Q5, Q6, Q7, Q8, Q9, R1, R10, R11, R12, R13, R14, R15, R16, R17, R18, R19, R2, R20, R21, R22, R23, R24, R25, R26, R27, R28, R3, R37, R38, R39, R4, R5, R6, R60, R65, R7, R8, R9, T1, TP2, TP3, U1, U2, U3, U5: moved to B.Cu
- C31, C33: value 10u -> 47p; moved to B.Cu
- C34: value 10u -> 10n; moved to B.Cu
- D6: value BAV99 -> GREEN_LED; footprint Package_TO_SOT_SMD:SOT-23 -> LED_SMD:LED_0805_2012Metric_Pad1.15x1.40mm_HandSolder; moved to B.Cu
- JP2, JP4, JP5: moved to F.Cu
- R34, R35: value 100 -> 5.1k; moved to B.Cu
- moved R35 165.5 mm to (67.3, 146.9), turned to 180 degrees
- moved R34 159.3 mm to (73.0, 146.8)
- moved C34 157.2 mm to (65.8, 154.8)
- moved C30 155.9 mm to (62.3, 159.5), turned to 90 degrees
- moved C31 155.3 mm to (66.5, 153.0), turned to 180 degrees
- moved C33 150.4 mm to (73.0, 153.0)
- moved D6 136.4 mm to (96.9, 151.3), turned to 180 degrees
- moved TP3 130.0 mm to (61.1, 164.0), turned to 180 degrees
- moved TP2 129.6 mm to (61.5, 155.0), turned to 180 degrees
- moved H4 118.1 mm to (55.0, 140.0)
- moved R12 101.4 mm to (78.8, 145.6), turned to 90 degrees
- moved R11 97.4 mm to (81.2, 145.6), turned to 90 degrees
- moved L4 96.9 mm to (81.0, 151.5)
- moved C45 95.2 mm to (90.2, 179.7)
- moved C7 94.3 mm to (78.3, 141.3), turned to 90 degrees
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Connections:
- net RX_5V renamed /Boost/RX
- C30 pad 1: 3V3 -> 5V
- C30 pad 2: GND -> Earth
- C31 pad 1: 5V -> Net-(C31-Pad1)
- C31 pad 2: GND -> Earth
- C33 pad 1: 5V -> Net-(C33-Pad1)
- C33 pad 2: GND -> Earth
- C34 pad 1: VREF -> Earth
- C34 pad 2: GND -> Net-(U4-V3)
- D6 pad 1: 5V -> Earth
- R2 pad 2: TX_5V -> /Boost/TX
- R34 pad 1: 5V -> Net-(J2-CC2)
- R34 pad 2: VREF -> Earth
- R35 pad 2: 5V -> Earth
- TP2 pad 1: VREF -> Earth
- TP3 pad 1: 3V3 -> 5V
Routing:
- added copper zone on B.Cu, net Earth
- removed copper zone on B.Cu, net (none)
- removed copper zone on F.Cu, net 3V3
- removed copper zone on B.Cu, net 5V
Other:
- board size 110 x 145 mm -> 110 x 60 mm

Commit message: SRF sch.
Parts:
- added C35: 47n, Capacitor_SMD:C_0603_1608Metric_Pad1.08x0.95mm_HandSolder, B.Cu at (187.4, 161.4)
- added C37: 47u, Capacitor_SMD:C_1206_3216Metric_Pad1.33x1.80mm_HandSolder, B.Cu at (204.6, 148.5)
- added C40: 47u, Capacitor_SMD:C_1206_3216Metric_Pad1.33x1.80mm_HandSolder, B.Cu at (204.6, 145.1)
- added C44: 10u, Capacitor_SMD:C_0603_1608Metric_Pad1.08x0.95mm_HandSolder, B.Cu at (187.4, 158.9)
- added C47: 10u, Capacitor_SMD:C_0603_1608Metric_Pad1.08x0.95mm_HandSolder, B.Cu at (187.4, 156.4)
- added C48: 10u, Capacitor_SMD:C_0603_1608Metric_Pad1.08x0.95mm_HandSolder, B.Cu at (187.4, 153.9)
- added C49: 10u, Capacitor_SMD:C_0603_1608Metric_Pad1.08x0.95mm_HandSolder, B.Cu at (187.4, 151.4)
- added C50: 10u, Capacitor_SMD:C_0603_1608Metric_Pad1.08x0.95mm_HandSolder, B.Cu at (191.7, 161.4)
- added C51: 10u, Capacitor_SMD:C_0603_1608Metric_Pad1.08x0.95mm_HandSolder, B.Cu at (191.7, 158.9)
- added C52: 10u, Capacitor_SMD:C_0603_1608Metric_Pad1.08x0.95mm_HandSolder, B.Cu at (191.7, 156.4)
- added C53: 10u, Capacitor_SMD:C_0603_1608Metric_Pad1.08x0.95mm_HandSolder, B.Cu at (191.7, 153.9)
- added C56: 100n, Capacitor_SMD:C_0603_1608Metric_Pad1.08x0.95mm_HandSolder, B.Cu at (191.7, 151.4)
- added C57: 10u, Capacitor_SMD:C_0603_1608Metric_Pad1.08x0.95mm_HandSolder, B.Cu at (196.1, 161.4)
- added C58: 10u, Capacitor_SMD:C_0603_1608Metric_Pad1.08x0.95mm_HandSolder, B.Cu at (196.1, 158.9)
- added C59: 10u, Capacitor_SMD:C_0603_1608Metric_Pad1.08x0.95mm_HandSolder, B.Cu at (196.1, 156.4)
- added D18: 1N5819WS, Diode_SMD:D_SOD-323, B.Cu at (199.5, 148.7)
- added D19: 1N5819WS, Diode_SMD:D_SOD-323, B.Cu at (199.5, 145.7)
- added D22: 1N5819WS, Diode_SMD:D_SOD-323, B.Cu at (199.5, 142.8)
- added D24: GREEN_LED, LED_SMD:LED_0805_2012Metric_Pad1.15x1.40mm_HandSolder, B.Cu at (193.6, 137.6)
- added L2: 220u, DC_load:L_Bourns_SRN6045TA, B.Cu at (201.3, 137.5)
- added Q1: MMBT5551L, Package_TO_SOT_SMD:SOT-23, B.Cu at (182.8, 160.3)
- added Q26: MMBT5551L, Package_TO_SOT_SMD:SOT-23, B.Cu at (182.8, 155.7)
- added Q27: MMBT5551L, Package_TO_SOT_SMD:SOT-23, B.Cu at (182.8, 151.0)
- added Q28: MMBT5551L, Package_TO_SOT_SMD:SOT-23, B.Cu at (182.8, 146.4)
- added Q29: MMBT5551L, Package_TO_SOT_SMD:SOT-23, B.Cu at (182.8, 141.8)
- added R36: 2.2k, Resistor_SMD:R_0603_1608Metric_Pad0.98x0.95mm_HandSolder, B.Cu at (196.1, 153.9)
- added R40: 1k, Resistor_SMD:R_0603_1608Metric_Pad0.98x0.95mm_HandSolder, B.Cu at (196.1, 151.4)
- added R41: 15k, Resistor_SMD:R_0603_1608Metric_Pad0.98x0.95mm_HandSolder, B.Cu at (200.4, 161.4)
- added R42: 10k, Resistor_SMD:R_0603_1608Metric_Pad0.98x0.95mm_HandSolder, B.Cu at (200.4, 158.9)
- added R47: 100m, Resistor_SMD:R_1206_3216Metric_Pad1.30x1.75mm_HandSolder, B.Cu at (188.2, 137.4)
- added R48: 100, Resistor_SMD:R_0603_1608Metric_Pad0.98x0.95mm_HandSolder, B.Cu at (200.4, 156.4)
- added R49: 1k, Resistor_SMD:R_0603_1608Metric_Pad0.98x0.95mm_HandSolder, B.Cu at (200.4, 153.9)
- added R52: 10k, Resistor_SMD:R_0603_1608Metric_Pad0.98x0.95mm_HandSolder, B.Cu at (200.4, 151.4)
- added T2: UMEC_UT20A13S, DC_load:UMEC_UT20A13S, B.Cu at (191.2, 144.6)
Connections:
- C45 pad 2: +VIN -> 5V
- C46 pad 2: +VIN -> 5V
- U5 pad 14: +VIN -> 5V

Commit message: SRF layout
Parts:
- added J1: Iso board connector, Connector_PinSocket_2.54mm:PinSocket_1x08_P2.54mm_Vertical, F.Cu at (55.0, 157.4)
- moved J12 83.4 mm to (76.8, 190.5), turned to -90 degrees
- moved D1 77.8 mm to (62.0, 185.9), turned to 180 degrees
- moved C27 76.4 mm to (64.7, 186.0), turned to 90 degrees
- moved R25 73.9 mm to (61.1, 182.4), turned to 90 degrees
- moved R1 72.6 mm to (70.1, 184.9), turned to 180 degrees
- moved Q7 72.2 mm to (63.9, 182.4), turned to 0 degrees
- moved D22 71.8 mm to (138.9, 181.3), turned to 90 degrees
- moved R18 71.4 mm to (73.6, 184.9), turned to 0 degrees
- moved D12 70.1 mm to (67.9, 182.4), turned to 0 degrees
- moved Q17 68.5 mm to (71.9, 182.4), turned to 180 degrees
- moved L2 67.7 mm to (139.4, 164.8), turned to 180 degrees
- moved R8 67.6 mm to (74.7, 182.4), turned to -90 degrees
- moved C59 66.3 mm to (135.5, 183.4), turned to 180 degrees
- moved C56 65.4 mm to (135.5, 184.9), turned to 180 degrees
- moved C58 64.8 mm to (135.5, 181.9), turned to 180 degrees
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
Commit message: Working on layout.
Parts:
- removed C44, C48, C50, C52: 10u, Capacitor_SMD:C_0603_1608Metric_Pad1.08x0.95mm_HandSolder
- added C36: 100n, Capacitor_SMD:C_0603_1608Metric_Pad1.08x0.95mm_HandSolder, B.Cu at (92.3, 164.9)
- added C38: 100n, Capacitor_SMD:C_0603_1608Metric_Pad1.08x0.95mm_HandSolder, B.Cu at (83.7, 181.9)
- added C39: 100n, Capacitor_SMD:C_0603_1608Metric_Pad1.08x0.95mm_HandSolder, B.Cu at (62.1, 179.8)
- added C41: 100n, Capacitor_SMD:C_0603_1608Metric_Pad1.08x0.95mm_HandSolder, B.Cu at (63.3, 166.1)
- added C42: 10u, Capacitor_SMD:C_0603_1608Metric_Pad1.08x0.95mm_HandSolder, B.Cu at (117.3, 188.9)
- added C43: 10u, Capacitor_SMD:C_0603_1608Metric_Pad1.08x0.95mm_HandSolder, B.Cu at (117.3, 185.6)
- added TP1: TestPoint, TestPoint:TestPoint_Pad_D2.0mm, F.Cu at (82.9, 139.2)
- added TP10: TestPoint, TestPoint:TestPoint_Pad_D2.0mm, F.Cu at (145.7, 163.1)
- added TP11: TestPoint, TestPoint:TestPoint_Pad_D2.0mm, F.Cu at (151.4, 159.7)
- added TP12: TestPoint, TestPoint:TestPoint_Pad_D2.0mm, F.Cu at (141.6, 181.4)
- added TP13: TestPoint, TestPoint:TestPoint_Pad_D2.0mm, F.Cu at (144.8, 181.4)
- added TP14: TestPoint, TestPoint:TestPoint_Pad_D2.0mm, F.Cu at (114.6, 165.0)
- added TP15: TestPoint, TestPoint:TestPoint_Pad_D2.0mm, F.Cu at (112.7, 160.6)
- added TP16: TestPoint, TestPoint:TestPoint_Pad_D2.0mm, F.Cu at (106.8, 165.6)
- added TP17: TestPoint, TestPoint:TestPoint_Pad_D2.0mm, F.Cu at (119.9, 137.8)
- added TP18: TestPoint, TestPoint:TestPoint_Pad_D2.0mm, F.Cu at (119.9, 140.8)
- added TP19: TestPoint, TestPoint:TestPoint_Pad_D2.0mm, F.Cu at (106.8, 160.6)
- added TP20: TestPoint, TestPoint:TestPoint_Pad_D2.0mm, F.Cu at (111.2, 191.8)
- added TP21: TestPoint, TestPoint:TestPoint_Pad_D2.0mm, F.Cu at (107.3, 191.8)
- added TP22: TestPoint, TestPoint:TestPoint_Pad_D2.0mm, F.Cu at (115.1, 191.8)
- added TP23: TestPoint, TestPoint:TestPoint_Pad_D2.0mm, F.Cu at (118.6, 163.2)
- added TP24: TestPoint, TestPoint:TestPoint_Pad_D2.0mm, F.Cu at (76.9, 160.5)
- added TP25: TestPoint, TestPoint:TestPoint_Pad_D2.0mm, F.Cu at (67.3, 160.5)
- added TP26: TestPoint, TestPoint:TestPoint_Pad_D2.0mm, F.Cu at (68.8, 187.2)
- added TP27: TestPoint, TestPoint:TestPoint_Pad_D2.0mm, F.Cu at (80.3, 187.2)
- added TP28: TestPoint, TestPoint:TestPoint_Pad_D2.0mm, F.Cu at (72.2, 160.5)
- added TP29: TestPoint, TestPoint:TestPoint_Pad_D2.0mm, F.Cu at (74.7, 187.2)
- added TP4: TestPoint, TestPoint:TestPoint_Pad_D2.0mm, F.Cu at (82.9, 147.8)
- added TP5: TestPoint, TestPoint:TestPoint_Pad_D2.0mm, F.Cu at (123.0, 159.3)
- added TP6: TestPoint, TestPoint:TestPoint_Pad_D2.0mm, F.Cu at (123.0, 162.3)
- added TP7: TestPoint, TestPoint:TestPoint_Pad_D2.0mm, F.Cu at (145.7, 157.0)
- added TP8: TestPoint, TestPoint:TestPoint_Pad_D2.0mm, F.Cu at (131.7, 170.2)
- added TP9: TestPoint, TestPoint:TestPoint_Pad_D2.0mm, F.Cu at (130.4, 164.8)
- JP1, JP3: moved to F.Cu
- moved C40 65.3 mm to (128.3, 165.9), turned to -90 degrees
- moved C37 63.0 mm to (128.3, 160.8), turned to 90 degrees
- moved D24 59.3 mm to (143.8, 184.7), turned to 180 degrees
- moved R49 57.0 mm to (130.4, 166.6), turned to -90 degrees
- moved R52 56.9 mm to (139.8, 184.3)
- moved D18 55.7 mm to (132.3, 166.5), turned to 90 degrees
- moved R40 49.9 mm to (134.2, 166.6), turned to -90 degrees
- moved R42 44.1 mm to (141.8, 160.5)
- moved C53 39.0 mm to (138.2, 155.8)
- moved C51 38.9 mm to (138.2, 159.0)
- moved C49 36.0 mm to (138.2, 160.6)
- moved C47 34.6 mm to (138.2, 157.4)
- moved R36 17.9 mm to (131.2, 164.0), turned to 0 degrees
- moved D19 17.1 mm to (131.3, 157.9)
- moved Q1 16.7 mm to (131.3, 161.1), turned to 90 degrees
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Connections:
- C10 pad 1: 11V -> Net-(D4-K)
- C11 pad 1: 11V -> Net-(D4-K)
- C12 pad 1: 11V -> Net-(D4-K)
- C47 pad 1: Net-(C47-Pad1) -> 5V
- C49 pad 1: Net-(C47-Pad1) -> 5V
- C51 pad 1: Net-(C47-Pad1) -> 5V
- C53 pad 1: Net-(C47-Pad1) -> 5V
- C9 pad 1: 11V -> Net-(D4-K)
- R28 pad 2: GND -> Earth
Routing:
- net 5V: track 0.00 -> 53.1 mm, vias 0 -> 9
- net /Boost/RX: track 0.00 -> 36.2 mm, vias 0 -> 1
- net Earth: track 0.00 -> 20.9 mm, vias 0 -> 19
- net /Boost/TX: track 0.00 -> 14.0 mm, vias 0 -> 1
- net TX_3V3: track 0.00 -> 13.8 mm, vias 0 -> 1
- net Net-(D11-A): track 0.00 -> 11.4 mm
- net Net-(Q4-B): track 0.00 -> 10.1 mm
- net 3V3: track 0.00 -> 9.67 mm, vias 0 -> 5
- net Net-(C33-Pad1): track 0.00 -> 9.53 mm
- net Net-(D13-A): track 0.00 -> 8.71 mm
- net Net-(Q7-B): track 0.00 -> 7.79 mm
- net GND: track 0.00 -> 7.68 mm, vias 0 -> 8
- net Net-(C31-Pad1): track 0.00 -> 6.60 mm
- net Net-(Q7-E): track 0.00 -> 3.42 mm
- net Net-(R3-Pad2): track 0.00 -> 2.68 mm
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- added copper zone on F.Cu, net Earth
- added copper zone on F.Cu, net GND
- removed copper zone on B.Cu, net Earth
- removed copper zone on B.Cu, net GND
