File: kicad/DC_load_isolation_module/isolated_supply.kicad_sch (KiCad schematic)
At the start: 43 parts, among them Q10 AO3400A, Q11 AO3400A, Q12 MMBT5551L, Q14 MMBT5401, Q15 MMBT5551L, Q16 MMBT5551L, Q8 MMBT5551L, Q9 MMBT5401

Commit message: Idk.
Parts:
- renumbered TR1 to TR2
Connections:
- net Earth: no longer C14.2, Q14.3 (C), R21.2
- net at Q10.3 (D), Q11.2 (S), TR2.1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: now also C14.2, Q14.3 (C), R21.2
Other:
- moved on the sheet: C10, C11, C12, C14, C15, C16, C17, C18, C19, C20, C21, C22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

Commit message: Schematic done.
Parts:
- added C13: 100p, Capacitor_SMD:C_0603_1608Metric_Pad1.08x0.95mm_HandSolder, symbol Device:C
- added C45: 100n, Capacitor_SMD:C_0603_1608Metric_Pad1.08x0.95mm_HandSolder, symbol Device:C
- added C46: 1u, Capacitor_SMD:C_0603_1608Metric_Pad1.08x0.95mm_HandSolder, symbol Device:C
- added D15: BAV99, Package_TO_SOT_SMD:SOT-23, symbol Diode:BAV99
- added R17, R39: 470k, Resistor_SMD:R_0603_1608Metric_Pad0.98x0.95mm_HandSolder, symbol Device:R
- added R24: 39k, Resistor_SMD:R_0603_1608Metric_Pad0.98x0.95mm_HandSolder, symbol Device:R
- added R27, R37: 100k, Resistor_SMD:R_0603_1608Metric_Pad0.98x0.95mm_HandSolder, symbol Device:R
- added U5: 74HC14D653, Package_SO:SOIC-14_3.9x8.7mm_P1.27mm, symbol 74xx:74HC14
- renumbered TR2 to TR1
Connections:
- net Earth: now also C13.1, C45.1, C46.1, U5.7 (GND); no longer C10.2, C11.2, C12.2, C9.2
- net GND: now also C10.2, C11.2, C12.2, C9.2, U5.1, U5.11, U5.3, U5.5
- net ~{BF_GATE}: now also U5.12
- net ~{TF_GATE}: now also R17.2, R24.1, R27.2, R37.2, R39.2, U5.13, U5.8
- new net: D15.2 (A), R27.1, R39.1
- new net: C13.2, D15.3 (K), R24.2, U5.9
- new net: D15.1 (K), R17.1, R37.1
- new net +VIN: C45.2, C46.2, U5.14 (VCC)
- no-connect marks 0 -> 4
Other:
- note added: "Bottom FET PWM gen"
- note added: "CLK generation"

Commit message: kk
Parts:
- removed TR1: TRANSF6, symbol Transformer:TRANSF6
- added T1: UMEC_UT20A13S, DC_load:UMEC_UT20A13S, symbol is:UMEC_UT20A13S
Connections:
- net at C14.2, Q10.3 (D), Q11.2 (S)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: now also T1.1 (AA), T1.2 (AA)
- net at C15.2, C16.2, C17.2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: now also T1.4 (AB)
- net at JP5.2 (B): now also T1.3 (AB)
- net at D8.2 (A), D9.1 (K): now also T1.6 (SA)
- net at D4.2 (A), D7.1 (K): now also T1.8 (SB)
- new net: T1.5 (SA), T1.7 (SB)
Other:
- moved on the sheet: C10, C11, C12, C14, C15, C16, C17, C18, C19, C20, C21, C22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

Commit message: Some placement.
Parts:
- added C32: 100n, Capacitor_SMD:C_0603_1608Metric_Pad1.08x0.95mm_HandSolder, symbol Device:C
Connections:
- net 12V: now also C32.1
- net Earth: now also C32.2
- net GND: now also U5.13, U5.9; no longer U5.1, U5.3
- net ~{BF_GATE}: now also U5.4; no longer U5.12
- net ~{TF_GATE}: now also U5.2, U5.3; no longer U5.13, U5.8
- net at C13.2, D15.3 (K), R24.2: now also U5.1; no longer U5.9

Commit message: M
Parts:
- added D16: GREEN_LED, LED_SMD:LED_0805_2012Metric_Pad1.15x1.40mm_HandSolder, symbol Device:LED
- added R33: 10k, Resistor_SMD:R_0603_1608Metric_Pad0.98x0.95mm_HandSolder, symbol Device:R
Connections:
- net 11V: now also R33.1
- net GND: now also D16.1 (K)
- net +VIN renamed 5V
- new net: D16.2 (A), R33.2
Other:
- moved on the sheet: C10, C11, C12, C14, C15, C16, C17, C18, C19, C20, C21, C22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

Commit message: Working on layout.
Parts:
- added C42, C43: 10u, Capacitor_SMD:C_0603_1608Metric_Pad1.08x0.95mm_HandSolder, symbol Device:C
- added TP14, TP15, TP16, TP17, TP18, TP19, TP20, TP21, TP22, TP23: TestPoint, TestPoint:TestPoint_Pad_D2.0mm, symbol Connector:TestPoint
Connections:
- net 11V: now also C42.1, C43.1, TP22.1; no longer C10.1, C11.1, C12.1, C9.1
- net Earth: now also TP17.1, TP19.1
- net GND: now also C42.2, C43.2, TP21.1
- net ~{TF_GATE}: now also TP18.1
- net at Q11.1 (G), R20.1, R21.1: now also TP14.1
- net at C14.2, Q10.3 (D), Q11.2 (S)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: now also TP15.1
- net at C15.2, C16.2, C17.2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: now also TP23.1
- net at Q10.1 (G), R15.1, R16.1: now also TP16.1
- net at D4.1 (K), D8.1 (K), JP4.1 (A)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: now also C10.1, C11.1, C12.1, C9.1, TP20.1
Other:
- moved on the sheet: C10, C11, C12, C9, D4, D8, JP4, L1

Commit message: Routing.
Connections:
- net Earth: now also U5.11, U5.13, U5.5, U5.9
- net GND: no longer U5.11, U5.13, U5.5, U5.9
Other:
- moved on the sheet: U5D, U5E, U5F
