File: kicad/DC_load_isolation_module/isolated_supply.kicad_sch (KiCad schematic)
At the start: 68 parts, among them Q10 AO3400A, Q11 AO3400A, Q12 MMBT5551L, Q14 MMBT5401, Q15 MMBT5551L, Q16 MMBT5551L, Q8 MMBT5551L, Q9 MMBT5401, T1 UMEC_UT20A13S, U5 74HC14D653

Commit message: Connectors fixed.
Connections:
- net 12V renamed 12V_PC
- net 5V renamed 5V_PC
Other:
- moved on the sheet: C10, C11, C12, C42, C43, C9, D4, D7, D8, D9, JP4, JP5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
