File: kicad/DC_load_isolation_module/boost.kicad_sch (KiCad schematic)
At the start: 28 parts, among them Q13 AO3400A, Q5 MMBT5401, Q6 MMBT5551L, U2 MC34063AD

Commit message: Schematic done.
Other:
- moved on the sheet: C4, C5, C6, C7, C8

Commit message: M
Parts:
- added C30: 10u, Capacitor_SMD:C_0603_1608Metric_Pad1.08x0.95mm_HandSolder, symbol Device:C
- added C31, C33: 47p, Capacitor_SMD:C_0603_1608Metric_Pad1.08x0.95mm_HandSolder, symbol Device:C
- added C34: 10n, Capacitor_SMD:C_0603_1608Metric_Pad1.08x0.95mm_HandSolder, symbol Device:C
- added D10, D6: GREEN_LED, LED_SMD:LED_0805_2012Metric_Pad1.15x1.40mm_HandSolder, symbol Device:LED
- added D17: 1N5819WS, Diode_SMD:D_SOD-323, symbol Diode:1N5819WS
- added J2: USB_C_Receptacle_USB2.0_16P, Connector_USB:USB_C_Receptacle_G-Switch_GT-USB-7010ASV, symbol Connector:USB_C_Receptacle_USB2.0_16P
- added R29, R30: 22, Resistor_SMD:R_0603_1608Metric_Pad0.98x0.95mm_HandSolder, symbol Device:R
- added R31: 10k, Resistor_SMD:R_0603_1608Metric_Pad0.98x0.95mm_HandSolder, symbol Device:R
- added R32: 1k, Resistor_SMD:R_0603_1608Metric_Pad0.98x0.95mm_HandSolder, symbol Device:R
- added R34, R35: 5.1k, Resistor_SMD:R_0603_1608Metric_Pad0.98x0.95mm_HandSolder, symbol Device:R
- added TP2, TP3: TestPoint, TestPoint:TestPoint_Pad_D2.0mm, symbol Connector:TestPoint
- added U4: CH340C, Package_SO:SOIC-16_3.9x9.9mm_P1.27mm, symbol DC_load:CH340C
Connections:
- net 12V: now also D17.1 (K), R31.1
- net 5V: now also C30.1, J2.A4 (VBUS), J2.A9 (VBUS), J2.B4 (VBUS), J2.B9 (VBUS), R32.1, TP3.1, U4.16 (VCC)
- net Earth: now also C30.2, C31.2, C33.2, C34.1, D10.1 (K), D6.1 (K), J2.A1 (GND), J2.A12 (GND), J2.B1 (GND), J2.B12 (GND), J2.S1 (SHIELD), R34.2, R35.2, TP2.1, U4.1 (GND)
- net at D5.2 (A), L4.2, Q13.3 (D): now also D17.2 (A)
- new net: R29.1, U4.5 (UD+)
- new net: C31.1, J2.A6 (D+), J2.B6 (D+), R29.2
- new net: R30.1, U4.6 (UD-)
- new net: C33.1, J2.A7 (D-), J2.B7 (D-), R30.2
- new net: J2.A5 (CC1), R35.1
- new net: D10.2 (A), R32.2
- new net: D6.2 (A), R31.2
- new net: J2.B5 (CC2), R34.1
- new net: C34.2, U4.4 (V3)
- new net RX: U4.3 (RXD)
- new net TX: U4.2 (TXD)
- no-connect marks 0 -> 9
Other:
- moved on the sheet: C2, C3, C4, C5, C54, C55, C6, C61, C62, C63, C7, C8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

Commit message: Working on layout.
Parts:
- added TP1, TP4, TP5, TP6: TestPoint, TestPoint:TestPoint_Pad_D2.0mm, symbol Connector:TestPoint
Connections:
- net 12V: now also TP6.1
- net Earth: now also TP5.1
- net at Q13.1 (G), R10.1, R38.1: now also TP1.1
- net at D17.2 (A), D5.2 (A), L4.2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: now also TP4.1
Other:
- moved on the sheet: L4

Commit message: Connectors fixed.
Connections:
- net 12V renamed 12V_PC
- net 5V renamed 5V_PC
Changed lines of the file:
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@@
 		)
 	)
-	(hierarchical_label "5V"
+	(hierarchical_label "5V_PC"
 		(shape output)
 		(at 52.07 27.94 0)
@@
 		)
 	)
-	(hierarchical_label "12V"
+	(hierarchical_label "12V_PC"
 		(shape output)
 		(at 246.38 110.49 0)
@@
 			)
 		)
-		(property "Value" "5V"
+		(property "Value" "5V_PC"
 			(at 138.43 117.348 0)
 			(effects
@@
 			)
 		)
-		(property "Value" "5V"
+		(property "Value" "5V_PC"
 			(at 67.31 76.2 0)
 			(effects
@@
 			)
 		)
-		(property "Value" "5V"
+		(property "Value" "5V_PC"
 			(at 45.72 102.87 0)
 			(effects
@@
 			)
 		)
-		(property "Value" "5V"
+		(property "Value" "5V_PC"
 			(at 115.57 121.92 0)
 			(effects
@@
 			)
 		)
-		(property "Value" "5V"
+		(property "Value" "5V_PC"
 			(at 182.88 38.1 0)
 			(effects
@@
 			)
 		)
-		(property "Value" "5V"
+		(property "Value" "5V_PC"
 			(at 49.53 20.32 0)
 			(effects
@@
 			)
 		)
-		(property "Value" "5V"
+		(property "Value" "5V_PC"
 			(at 25.4 74.93 0)
 			(effects
@@
 			)
 		)
-		(property "Value" "12V"
+		(property "Value" "12V_PC"
 			(at 262.89 107.95 0)
 			(effects
@@
 			)
 		)
-		(property "Value" "5V"
+		(property "Value" "5V_PC"
 			(at 121.92 31.75 0)
 			(effects
@@
 			)
 		)
-		(property "Value" "12V"
+		(property "Value" "12V_PC"
 			(at 231.14 102.87 0)
 			(effects
