File: kicad/DC_load_isolation_module/DC_load_isolation_module.kicad_sch (KiCad schematic)
At the start: 39 parts, among them J6 USB_B, Q1 MMBT5401, Q2 MMBT5401, Q7 MMBT5551L, U14 AMS1117-3.3, U17 CH340C, U18 TL431DBZ, U3 LTV-817S

Commit message: up
Parts:
- removed R50: 100, Resistor_SMD:R_0603_1608Metric_Pad0.98x0.95mm_HandSolder, symbol Device:R
- added C1: 100n, Capacitor_SMD:C_0603_1608Metric_Pad1.08x0.95mm_HandSolder, symbol Device:C
- added D2: BAV99, Package_TO_SOT_SMD:SOT-23, symbol Diode:BAV99
- added Q3: MMBT5401, Package_TO_SOT_SMD:SOT-23, symbol Transistor_BJT:MMBT3906
- added Q4: MMBT5551L, Package_TO_SOT_SMD:SOT-23, symbol Transistor_BJT:MMBT5551L
- added R1, R6: 1k, Resistor_SMD:R_0603_1608Metric_Pad0.98x0.95mm_HandSolder, symbol Device:R
- added R2, R4: 100, Resistor_SMD:R_0603_1608Metric_Pad0.98x0.95mm_HandSolder, symbol Device:R
- added R3, R5: 220, Resistor_SMD:R_0603_1608Metric_Pad0.98x0.95mm_HandSolder, symbol Device:R
- added R7: 10k, Resistor_SMD:R_0603_1608Metric_Pad0.98x0.95mm_HandSolder, symbol Device:R
- added U1: LTV-817S, Package_DIP:SMDIP-4_W9.53mm, symbol Isolator:LTV-817S
Connections:
- net 3V3: now also R8.1, R1.1, R7.1; no longer U17.16 (VCC)
- net 5V: now also U17.16 (VCC), R3.1, R6.1; no longer R8.1
- net GND: now also C1.1, D2.2 (A), Q3.3 (C), U1.3
- net TX: now also U17.2 (TXD), R2.2, R4.2
- net at Q2.1 (B): now also R2.1
- net at U3.1: now also R3.2
- net TX_3V3: now reaches Q7.3 (C)
- net TX_3V3: now also R1.2
- new net: Q3.1 (B), R4.1
- new net: C1.2, D2.1 (K), Q4.1 (B), R7.2
- new net: Q4.2 (E), U1.4
- new net: Q3.2 (E), U1.2
- new net: R5.2, U1.1
- new net RX_5V: Q4.3 (C), R6.2
- no-connect marks 8 -> 10
Other:
- moved on the sheet: C69, D1, H1, H2, H3, H4, Q2, Q7, R8, U3

Commit message: Sim, comp, power.
Parts:
- removed C1, C69: 100n, Capacitor_SMD:C_0603_1608Metric_Pad1.08x0.95mm_HandSolder, symbol Device:C
- removed D1, D2: BAV99, Package_TO_SOT_SMD:SOT-23, symbol Diode:BAV99
- removed Q2, Q3: MMBT5401, Package_TO_SOT_SMD:SOT-23, symbol Transistor_BJT:MMBT3906
- removed Q4, Q7: MMBT5551L, Package_TO_SOT_SMD:SOT-23, symbol Transistor_BJT:MMBT5551L
- removed R1, R6: 1k, Resistor_SMD:R_0603_1608Metric_Pad0.98x0.95mm_HandSolder, symbol Device:R
- removed R2, R4: 100, Resistor_SMD:R_0603_1608Metric_Pad0.98x0.95mm_HandSolder, symbol Device:R
- removed R3, R5: 220, Resistor_SMD:R_0603_1608Metric_Pad0.98x0.95mm_HandSolder, symbol Device:R
- removed R7, R8: 10k, Resistor_SMD:R_0603_1608Metric_Pad0.98x0.95mm_HandSolder, symbol Device:R
- removed U1, U3: LTV-817S, Package_DIP:SMDIP-4_W9.53mm, symbol Isolator:LTV-817S
- added C2, C3: 220p, Capacitor_SMD:C_0603_1608Metric_Pad1.08x0.95mm_HandSolder, symbol Device:C
- added C4, C55: 100n, Capacitor_SMD:C_0603_1608Metric_Pad1.08x0.95mm_HandSolder, symbol Device:C
- added C5, C54, C6, C61, C62, C63, C7, C8: 10u, Capacitor_SMD:C_0603_1608Metric_Pad1.08x0.95mm_HandSolder, symbol Device:C
- added D5: 1N5819WS, Diode_SMD:D_SOD-323, symbol Diode:1N5819WS
- added JP1, JP3: Jumper_2_Open, Jumper:SolderJumper-2_P1.3mm_Open_RoundedPad1.0x1.5mm, symbol Jumper:Jumper_2_Open
- added L4: 220u, DC_load:L_Bourns_SRN6045TA, symbol solar_push_pull_sym_lib:SRN6045HA-4R7Y
- added Q13: AO3400A, Package_TO_SOT_SMD:SOT-23, symbol Transistor_FET:AO3400A
- added Q5: MMBT5401, Package_TO_SOT_SMD:SOT-23, symbol Transistor_BJT:MMBT3906
- added Q6: MMBT5551L, Package_TO_SOT_SMD:SOT-23, symbol Transistor_BJT:MMBT5551L
- added R10: 10, Resistor_SMD:R_0603_1608Metric_Pad0.98x0.95mm_HandSolder, symbol Device:R
- added R11, R12: 100m, Resistor_SMD:R_1206_3216Metric_Pad1.30x1.75mm_HandSolder, symbol Device:R
- added R13, R38: 100k, Resistor_SMD:R_0603_1608Metric_Pad0.98x0.95mm_HandSolder, symbol Device:R
- added R60: 1Meg, Resistor_SMD:R_0603_1608Metric_Pad0.98x0.95mm_HandSolder, symbol Device:R
- added R65: 10k, Resistor_SMD:R_0603_1608Metric_Pad0.98x0.95mm_HandSolder, symbol Device:R
- added R9: 1k, Resistor_SMD:R_0603_1608Metric_Pad0.98x0.95mm_HandSolder, symbol Device:R
- added U2: MC34063AD, Package_SO:SOIC-8_3.9x4.9mm_P1.27mm, symbol Regulator_Switching:MC34063AD
Connections:
- net 5V: now also C4.1, C5.1, C6.1, C7.1, C8.1, JP1.1 (A), Q6.3 (C), R11.2, R12.2, U2.1 (SwC), U2.6 (Vin), U2.8 (DC)
- net GND: no longer C42.2, C43.2, C44.1, C48.1, C57.2, J6.4 (GND), J6.5 (Shield), TP5.1, U17.1 (GND)
- new net: Q13.1 (G), R10.1, R38.1
- new net: JP1.2 (B), L4.1, R11.1, R12.1, U2.7 (Ipk)
- new net: D5.2 (A), L4.2, Q13.3 (D)
- new net: C2.1, C3.1, U2.3 (TC)
- new net: JP3.1 (A), Q5.1 (B), Q6.1 (B), R9.1, U2.2 (SwE)
- new net: JP3.2 (B), Q5.2 (E), Q6.2 (E), R10.2
- new net 12V: C54.1, C55.1, C61.1, C62.1, C63.1, D5.1 (K), R13.1, R60.1
- new net BFB: R13.2, R60.2, R65.1, U2.5 (Vfb)
- new net Earth: C2.2, C3.2, C4.2, C42.2, C43.2, C44.1, C48.1, C5.2, C54.2, C55.2, C57.2, C6.2, C61.2, C62.2, C63.2, C7.2, C8.2, J6.4 (GND), J6.5 (Shield), Q13.2 (S), Q5.3 (C), R38.2, R65.2, R9.2, TP5.1, U17.1 (GND), U2.4 (GND)
- no-connect marks 10 -> 8
Other:
- added sheet Isolated logic (isolated_logic.kicad_sch)
- added sheet Isolated supply (isolated_supply.kicad_sch)
- moved on the sheet: C57, TP5

Commit message: Idk.
Parts:
- removed C2, C3: 220p, Capacitor_SMD:C_0603_1608Metric_Pad1.08x0.95mm_HandSolder, symbol Device:C
- removed C4, C55: 100n, Capacitor_SMD:C_0603_1608Metric_Pad1.08x0.95mm_HandSolder, symbol Device:C
- removed C5, C54, C6, C61, C62, C63, C7, C8: 10u, Capacitor_SMD:C_0603_1608Metric_Pad1.08x0.95mm_HandSolder, symbol Device:C
- removed D5: 1N5819WS, Diode_SMD:D_SOD-323, symbol Diode:1N5819WS
- removed JP1, JP3: Jumper_2_Open, Jumper:SolderJumper-2_P1.3mm_Open_RoundedPad1.0x1.5mm, symbol Jumper:Jumper_2_Open
- removed L4: 220u, DC_load:L_Bourns_SRN6045TA, symbol solar_push_pull_sym_lib:SRN6045HA-4R7Y
- removed Q13: AO3400A, Package_TO_SOT_SMD:SOT-23, symbol Transistor_FET:AO3400A
- removed Q5: MMBT5401, Package_TO_SOT_SMD:SOT-23, symbol Transistor_BJT:MMBT3906
- removed Q6: MMBT5551L, Package_TO_SOT_SMD:SOT-23, symbol Transistor_BJT:MMBT5551L
- removed R10: 10, Resistor_SMD:R_0603_1608Metric_Pad0.98x0.95mm_HandSolder, symbol Device:R
- removed R11, R12: 100m, Resistor_SMD:R_1206_3216Metric_Pad1.30x1.75mm_HandSolder, symbol Device:R
- removed R13, R38: 100k, Resistor_SMD:R_0603_1608Metric_Pad0.98x0.95mm_HandSolder, symbol Device:R
- removed R60: 1Meg, Resistor_SMD:R_0603_1608Metric_Pad0.98x0.95mm_HandSolder, symbol Device:R
- removed R65: 10k, Resistor_SMD:R_0603_1608Metric_Pad0.98x0.95mm_HandSolder, symbol Device:R
- removed R9: 1k, Resistor_SMD:R_0603_1608Metric_Pad0.98x0.95mm_HandSolder, symbol Device:R
- removed U2: MC34063AD, Package_SO:SOIC-8_3.9x4.9mm_P1.27mm, symbol Regulator_Switching:MC34063AD
Other:
- added sheet Boost (boost.kicad_sch)

Commit message: M
Parts:
- removed C30, C31, C33, C34, C35, C57: 10u, Capacitor_SMD:C_0603_1608Metric_Pad1.08x0.95mm_HandSolder, symbol Device:C
- removed C42, C43: 47p, Capacitor_SMD:C_0603_1608Metric_Pad1.08x0.95mm_HandSolder, symbol Device:C
- removed C44: 10n, Capacitor_SMD:C_0603_1608Metric_Pad1.08x0.95mm_HandSolder, symbol Device:C
- removed C48: 100n, Capacitor_SMD:C_0603_1608Metric_Pad1.08x0.95mm_HandSolder, symbol Device:C
- removed D6: BAV99, Package_TO_SOT_SMD:SOT-23, symbol Diode:BAV99
- removed J6: USB_B, DC_load:62910416121, symbol Connector:USB_B
- removed Q1: MMBT5401, Package_TO_SOT_SMD:SOT-23, symbol Transistor_BJT:MMBT3906
- removed R34, R35: 100, Resistor_SMD:R_0603_1608Metric_Pad0.98x0.95mm_HandSolder, symbol Device:R
- removed R48, R49: 22, Resistor_SMD:R_0603_1608Metric_Pad0.98x0.95mm_HandSolder, symbol Device:R
- removed R56, R58: 10k, Resistor_SMD:R_0603_1608Metric_Pad0.98x0.95mm_HandSolder, symbol Device:R
- removed R57: 49.9k, Resistor_SMD:R_0603_1608Metric_Pad0.98x0.95mm_HandSolder, symbol Device:R
- removed TP1, TP2, TP3, TP4, TP5: TestPoint, TestPoint:TestPoint_Pad_D2.0mm, symbol Connector:TestPoint
- removed U14: AMS1117-3.3, Package_TO_SOT_SMD:SOT-223-3_TabPin2, symbol Regulator_Linear:AMS1117-3.3
- removed U17: CH340C, Package_SO:SOIC-16_3.9x9.9mm_P1.27mm, symbol DC_load:CH340C
- removed U18: TL431DBZ, Package_TO_SOT_SMD:SOT-23, symbol Reference_Voltage:TL431DBZ
Connections:
- no-connect marks 8 -> 0
Other:
- sheet Boost ports: added 12V, 5V, RX, TX; removed none
- sheet Isolated logic ports: added RX, TX; removed none
- sheet Isolated supply ports: added 12V, 5V; removed none
- note removed: "Linear regulator"
- note removed: "Voltage reference"
- title: DC load -> DC load isolation module
- moved on the sheet: H1, H2, H3, H4

Commit message: SRF sch.
Other:
- added sheet Self resonating flyback (srf.kicad_sch)
Changed lines of the file:
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@@
 	(wire
 		(pts
-			(xy 80.01 27.94) (xy 93.98 27.94)
+			(xy 80.01 43.18) (xy 93.98 43.18)
 		)
 		(stroke
@@
 	(wire
 		(pts
-			(xy 80.01 25.4) (xy 93.98 25.4)
+			(xy 80.01 45.72) (xy 93.98 45.72)
 		)
 		(stroke
@@
 	)
 	(sheet
-		(at 93.98 46.99)
-		(size 35.56 26.67)
+		(at 93.98 62.23)
+		(size 35.56 11.43)
 		(exclude_from_sim no)
 		(in_bom yes)
@@
 		)
 		(property "Sheetname" "Isolated logic"
-			(at 93.98 46.2784 0)
+			(at 93.98 61.5184 0)
 			(effects
 				(font
@@
 	)
 	(sheet
-		(at 93.98 22.86)
-		(size 35.56 16.51)
+		(at 93.98 40.64)
+		(size 35.56 15.24)
 		(exclude_from_sim no)
 		(in_bom yes)
@@
 		)
 		(property "Sheetname" "Isolated supply"
+			(at 93.98 39.9284 0)
+			(effects
+				(font
+					(size 1.27 1.27)
+				)
+				(justify left bottom)
+			)
+		)
+		(property "Sheetfile" "isolated_supply.kicad_sch"
+			(at 93.98 56.4646 0)
+			(effects
+				(font
+					(size 1.27 1.27)
+				)
+				(justify left top)
+			)
+		)
+		(pin "5V" input
+			(at 93.98 45.72 180)
+			(effects
+				(font
+					(size 1.27 1.27)
+				)
+				(justify left)
+			)
+		)
+		(pin "12V" input
+			(at 93.98 43.18 180)
+			(effects
+				(font
+					(size 1.27 1.27)
+				)
+				(justify left)
+			)
+		)
+		(instances
+			(project "DC_load_isolation_module"
+				(path "/ce255642-b081-42cc-af02-07a78c62b42e"
+					(page "3")
+				)
+			)
+		)
+	)
+	(sheet
+		(at 93.98 22.86)
+		(size 35.56 11.43)
+		(exclude_from_sim no)
+		(in_bom yes)
+		(on_board yes)
+		(dnp no)
+		(fields_autoplaced yes)
+		(stroke
+			(width 0.1524)
+			(type solid)
+		)
+		(fill
+			(color 0 0 0 0.0000)
+		)
+		(property "Sheetname" "Self resonating flyback"
 			(at 93.98 22.1484 0)
 			(effects
@@
 			)
 		)
-		(property "Sheetfile" "isolated_supply.kicad_sch"
-			(at 93.98 39.9546 0)
+		(property "Sheetfile" "srf.kicad_sch"
+			(at 93.98 34.8746 0)
 			(effects
 				(font
@@
 			)
 		)
-		(pin "5V" input
-			(at 93.98 27.94 180)
-			(effects
-				(font
-					(size 1.27 1.27)
-				)
-				(justify left)
-			)
-		)
-		(pin "12V" input
-			(at 93.98 25.4 180)
-			(effects
-				(font
-					(size 1.27 1.27)
-				)
-				(justify left)
-			)
-		)
 		(instances
 			(project "DC_load_isolation_module"
 				(path "/ce255642-b081-42cc-af02-07a78c62b42e"
-					(page "3")
+					(page "5")
 				)
 			)
@@
 		)
 		(pin "12V" output
-			(at 80.01 25.4 0)
+			(at 80.01 43.18 0)
 			(effects
 				(font
@@
 		)
 		(pin "5V" output
-			(at 80.01 27.94 0)
-			(effects
-				(font
+			(at 80.01 45.72 0)
+			(effects
+				(font

Commit message: SRF layout
Parts:
- added J1, J12: Iso board connector, Connector_PinSocket_2.54mm:PinSocket_1x08_P2.54mm_Vertical, symbol Connector:Conn_01x08_Socket
Connections:
- new net 12V: J1.1 (Pin_1)
- new net 12V_EXT: J12.6 (Pin_6)
- new net 3V3: J12.2 (Pin_2)
- new net 5V_EXT: J12.7 (Pin_7)
- new net Earth: J12.8 (Pin_8)
- new net GND: J1.8 (Pin_8), J12.5 (Pin_5)
- new net RX_3V3: J12.3 (Pin_3)
- new net TX_3V3: J12.4 (Pin_4)
- new net VCC: J12.1 (Pin_1)
Other:
- sheet Self resonating flyback ports: added 5V; removed none
- moved on the sheet: H1, H2, H3, H4

Commit message: Connectors fixed.
Parts:
- added J3: Conn_01x03_Pin, Connector_PinHeader_2.54mm:PinHeader_1x03_P2.54mm_Vertical, symbol Connector:Conn_01x03_Pin
- J1: value Iso board connector -> PC referenced connector
- J12: value Iso board connector -> Load referenced connector
Connections:
- net 12V_EXT is gone; now on net GND: J12.6 (Pin_6)
- net 5V_EXT is gone; now on net 3V3: J12.7 (Pin_7)
- net 3V3: no longer J12.2 (Pin_2)
- net Earth: now also J1.2 (Pin_2), J1.4 (Pin_4); no longer J12.8 (Pin_8)
- net GND: now also J12.2 (Pin_2), J12.4 (Pin_4), J12.8 (Pin_8); no longer J1.8 (Pin_8), J12.5 (Pin_5)
- net TX_3V3: now also J12.5 (Pin_5); no longer J12.4 (Pin_4)
- net VCC: now also J3.2 (Pin_2)
- net 5V_PC_PC: now reaches J1.3 (Pin_3)
- net 12V renamed 12V_PC
- new net Isolated supply/11V: J3.1 (Pin_1)
- new net Self resonating flyback/11V_SRF: J3.3 (Pin_3)
- no-connect marks 0 -> 4
Other:
- sheet Boost ports: added 12V_PC, 5V_PC; removed 12V, 5V
- sheet Isolated supply ports: added 11V, 12V_PC, 5V_PC; removed 12V, 5V
- sheet Self resonating flyback ports: added 11V_SRF, 5V_PC; removed 5V
- moved on the sheet: J1, J12

Commit message: Iso module almost done.
Connections:
- net 5V_PC_PC renamed 5V_PC
Changed lines of the file:
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@@
 		(on_board yes)
 		(dnp no)
-		(fields_autoplaced yes)
 		(property "Reference" "#PWR0177"
 			(at 149.86 48.26 0)
@@
 			)
 		)
-		(property "Value" "5V_PC_PC"
-			(at 142.24 48.2599 90)
+		(property "Value" "5V_PC"
+			(at 138.43 48.26 90)
 			(effects
 				(font
 					(size 1.27 1.27)
 				)
-				(justify left)
 			)
 		)
