File: kicad/DC_load_isolation_module/srf.kicad_sch (KiCad schematic)
At the start: 34 parts, among them Q1 MMBT5551L, Q26 MMBT5551L, Q27 MMBT5551L, Q28 MMBT5551L, Q29 MMBT5551L, T2 UMEC_UT20A13S

Commit message: Working on layout.
Parts:
- removed C44, C48, C50, C52: 10u, Capacitor_SMD:C_0603_1608Metric_Pad1.08x0.95mm_HandSolder, symbol Device:C
- added TP10, TP11, TP12, TP13, TP7, TP8, TP9: TestPoint, TestPoint:TestPoint_Pad_D2.0mm, symbol Connector:TestPoint
Connections:
- net 11V_SRF: now also TP12.1
- net 5V: now also C47.1, C49.1, C51.1, C53.1
- net GND: now also TP13.1
- net at D18.1 (K), R40.2, T2.1 (AA): now also TP8.1
- net at L2.1, Q26.3 (C), Q27.3 (C)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: now also TP10.1
- net at C35.1, D19.1 (K), Q1.3 (C)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: now also TP7.1
- net at Q26.2 (E), Q27.2 (E), Q28.2 (E)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: now also TP11.1
- net at C37.1, C40.1, D18.2 (A)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: now also TP9.1
Other:
- moved on the sheet: C47, C49, C51, C53

Commit message: Connectors fixed.
Connections:
- net 5V renamed 5V_PC
Other:
- moved on the sheet: D24, R52
Changed lines of the file:
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@@
 	)
 	(junction
+		(at 152.4 101.6)
+		(diameter 0)
+		(color 0 0 0 0)
+	)
+	(junction
 		(at 34.29 91.44)
 		(diameter 0)
@@
 	(wire
 		(pts
-			(xy 156.21 119.38) (xy 156.21 121.92)
+			(xy 152.4 116.84) (xy 152.4 124.46)
 		)
 		(stroke
@@
 	(wire
 		(pts
-			(xy 156.21 109.22) (xy 156.21 111.76)
+			(xy 152.4 101.6) (xy 152.4 109.22)
 		)
 		(stroke
@@
 	(wire
 		(pts
-			(xy 146.05 101.6) (xy 146.05 99.06)
-		)
-		(stroke
-			(width 0)
-			(type default)
-		)
-	)
-	(wire
-		(pts
 			(xy 24.13 27.94) (xy 24.13 35.56)
 		)
@@
 	(wire
 		(pts
+			(xy 146.05 101.6) (xy 152.4 101.6)
+		)
+		(stroke
+			(width 0)
+			(type default)
+		)
+	)
+	(wire
+		(pts
 			(xy 46.99 35.56) (xy 67.31 35.56)
 		)
@@
 	(wire
 		(pts
+			(xy 152.4 101.6) (xy 156.21 101.6)
+		)
+		(stroke
+			(width 0)
+			(type default)
+		)
+	)
+	(wire
+		(pts
 			(xy 38.1 49.53) (xy 43.18 49.53)
 		)
@@
 	(wire
 		(pts
-			(xy 156.21 132.08) (xy 156.21 129.54)
+			(xy 152.4 138.43) (xy 152.4 132.08)
 		)
 		(stroke
@@
 		)
 	)
-	(hierarchical_label "5V"
-		(shape input)
-		(at 31.75 91.44 180)
+	(hierarchical_label "11V_SRF"
+		(shape output)
+		(at 156.21 101.6 0)
 		(effects
 			(font
 				(size 1.27 1.27)
 			)
-			(justify right)
+			(justify left)
 		)
 	)
-	(symbol
-		(lib_id "power:+5V")
-		(at 146.05 99.06 0)
-		(unit 1)
-		(exclude_from_sim no)
-		(in_bom yes)
-		(on_board yes)
-		(dnp no)
-		(fields_autoplaced yes)
-		(property "Reference" "#PWR0134"
-			(at 146.05 102.87 0)
-			(effects
-				(font
-					(size 1.27 1.27)
-				)
-				(hide yes)
-			)
-		)
-		(property "Value" "11V_SRF"
-			(at 146.05 93.98 0)
-			(effects
-				(font
-					(size 1.27 1.27)
-				)
-			)
-		)
-		(property "Footprint" ""
-			(at 146.05 99.06 0)
-			(effects
-				(font
-					(size 1.27 1.27)
-				)
-				(hide yes)
-			)
-		)
-		(property "Datasheet" ""
-			(at 146.05 99.06 0)
-			(effects
-				(font
-					(size 1.27 1.27)
-				)
-				(hide yes)
-			)
-		)
-		(property "Description" "Power symbol creates a global label with name \"+5V\""
-			(at 146.05 99.06 0)
-			(effects
-				(font
-					(size 1.27 1.27)
-				)
-				(hide yes)
-			)
-		)
-		(pin "1"
-		)
-		(instances
-			(project "DC_load_isolation_module"
-				(path "/ce255642-b081-42cc-af02-07a78c62b42e/acb3fb6f-8a66-4a1f-8458-7972da3ba4df"
-					(reference "#PWR0134")
-					(unit 1)
-				)
+	(hierarchical_label "5V_PC"
+		(shape input)
+		(at 31.75 91.44 180)
+		(effects
+			(font
+				(size 1.27 1.27)
 			)
+			(justify right)
 		)
 	)
@@
 	)
 	(symbol
-		(lib_id "power:+5V")
-		(at 156.21 109.22 0)
-		(mirror y)
-		(unit 1)
-		(exclude_from_sim no)
-		(in_bom yes)
-		(on_board yes)
-		(dnp no)
-		(fields_autoplaced yes)
-		(property "Reference" "#PWR0103"
-			(at 156.21 113.03 0)
-			(effects
-				(font
-					(size 1.27 1.27)
-				)
-				(hide yes)
-			)
-		)
-		(property "Value" "11V_SRF"
-			(at 156.21 104.14 0)
-			(effects
-				(font
-					(size 1.27 1.27)
-				)
-			)
-		)
-		(property "Footprint" ""
-			(at 156.21 109.22 0)
-			(effects
-				(font
-					(size 1.27 1.27)
-				)
-				(hide yes)
-			)
-		)
-		(property "Datasheet" ""
-			(at 156.21 109.22 0)
-			(effects
-				(font
-					(size 1.27 1.27)
-				)
-				(hide yes)
-			)
-		)
-		(property "Description" "Power symbol creates a global label with name \"+5V\""
-			(at 156.21 109.22 0)
-			(effects
-				(font
-					(size 1.27 1.27)
-				)
-				(hide yes)
-			)
-		)
-		(pin "1"
-		)
-		(instances
-			(project "DC_load_isolation_module"
-				(path "/ce255642-b081-42cc-af02-07a78c62b42e/acb3fb6f-8a66-4a1f-8458-7972da3ba4df"
-					(reference "#PWR0103")
-					(unit 1)
-				)
-			)
-		)
-	)
-	(symbol
 		(lib_id "power:GND")
 		(at 115.57 138.43 0)
@@
 			)
 		)
-		(property "Value" "5V"
+		(property "Value" "5V_PC"
 			(at 59.69 85.09 0)
 			(effects
@@
 	(symbol
 		(lib_id "Device:R")
-		(at 156.21 115.57 0)
+		(at 152.4 113.03 0)
 		(unit 1)
 		(exclude_from_sim no)
@@
 		(dnp no)
 		(property "Reference" "R52"
-			(at 158.75 114.2999 0)
+			(at 154.94 111.7599 0)
 			(effects
 				(font
@@
 		)
 		(property "Value" "10k"
-			(at 158.75 116.8399 0)
+			(at 154.94 114.2999 0)
 			(effects
 				(font
@@
 		)
 		(property "Footprint" "Resistor_SMD:R_0603_1608Metric_Pad0.98x0.95mm_HandSolder"
-			(at 154.432 115.57 90)
+			(at 150.622 113.03 90)
 			(effects
 				(font
@@
 		)
 		(property "Datasheet" "~"
-			(at 156.21 115.57 0)
+			(at 152.4 113.03 0)
 			(effects
 				(font
@@
 		)
 		(property "Description" ""
-			(at 156.21 115.57 0)
+			(at 152.4 113.03 0)
 			(effects
 				(font
@@
 		)
 		(property "LCSC" "C25804"
-			(at 156.21 115.57 0)
+			(at 152.4 113.03 0)
 			(effects
 				(font
@@
 	(symbol
 		(lib_id "power:GND")
-		(at 156.21 132.08 0)
+		(at 152.4 138.43 0)
 		(unit 1)
 		(exclude_from_sim no)
@@
 		(fields_autoplaced yes)
 		(property "Reference" "#PWR0137"
-			(at 156.21 138.43 0)
+			(at 152.4 144.78 0)
 			(effects
 				(font
@@
 		)
 		(property "Value" "GND"
-			(at 156.21 137.16 0)
+			(at 152.4 143.51 0)
 			(effects
 				(font
@@
 		)
 		(property "Footprint" ""
-			(at 156.21 132.08 0)
+			(at 152.4 138.43 0)
 			(effects
 				(font
@@
 		)
 		(property "Datasheet" ""
-			(at 156.21 132.08 0)
+			(at 152.4 138.43 0)
 			(effects
 				(font
@@
 		)
 		(property "Description" "Power symbol creates a global label with name \"GND\" , ground"
-			(at 156.21 132.08 0)
+			(at 152.4 138.43 0)
 			(effects
 				(font
@@
 	(symbol
 		(lib_id "Device:LED")
-		(at 156.21 125.73 90)
+		(at 152.4 128.27 90)
 		(unit 1)
 		(exclude_from_sim no)
@@
 		(fields_autoplaced yes)
 		(property "Reference" "D24"
-			(at 160.02 126.0474 90)
+			(at 156.21 128.5874 90)
 			(effects
 				(font
@@
 		)
 		(property "Value" "GREEN_LED"
-			(at 160.02 128.5874 90)
+			(at 156.21 131.1274 90)
 			(effects
 				(font
@@
 		)
 		(property "Footprint" "LED_SMD:LED_0805_2012Metric_Pad1.15x1.40mm_HandSolder"
-			(at 156.21 125.73 0)
+			(at 152.4 128.27 0)
 			(effects
 				(font
@@
 		)
 		(property "Datasheet" "~"
-			(at 156.21 125.73 0)
+			(at 152.4 128.27 0)
 			(effects
 				(font
@@
 		)
 		(property "Description" "Light emitting diode"
-			(at 156.21 125.73 0)
+			(at 152.4 128.27 0)
 			(effects
 				(font
@@
 		)
 		(property "Sim.Pins" "1=K 2=A"
-			(at 156.21 125.73 0)
+			(at 152.4 128.27 0)
 			(effects
 				(font
@@
 		)
 		(property "LCSC" "C2297"
-			(at 156.21 125.73 90)
+			(at 152.4 128.27 90)
 			(effects
 				(font

Commit message: Fixes
Parts:
- added R43, R44, R45: 100m, Resistor_SMD:R_1206_3216Metric_Pad1.30x1.75mm_HandSolder, symbol Device:R
- added R46, R50, R51: 100, Resistor_SMD:R_0603_1608Metric_Pad0.98x0.95mm_HandSolder, symbol Device:R
Connections:
- net at C35.1, D19.1 (K), Q1.3 (C)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: now also R46.2, R50.2, R51.2; no longer Q26.1 (B), Q27.1 (B), Q28.1 (B)
- net at R47.2, R48.1, TP11.1: now also R43.1, R44.1, R45.1; no longer Q26.2 (E), Q27.2 (E), Q28.2 (E)
- new net: Q28.2 (E), R43.2
- new net: Q27.1 (B), R46.1
- new net: Q26.2 (E), R44.2
- new net: Q26.1 (B), R50.1
- new net: Q27.2 (E), R45.2
- new net: Q28.1 (B), R51.1
Other:
- moved on the sheet: Q29, R47, R48, TP11

Commit message: kfsald
Other:
- moved on the sheet: R43
Changed lines of the file:
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@@
 	(symbol
 		(lib_id "Device:R")
-		(at 95.25 140.97 180)
+		(at 95.25 140.97 0)
+		(mirror x)
 		(unit 1)
 		(exclude_from_sim no)
@@
 		(dnp no)
 		(property "Reference" "R43"
-			(at 90.17 139.7 0)
+			(at 92.71 137.16 0)
 			(effects
 				(font
@@
 		)
 		(property "Value" "100m"
-			(at 90.17 142.24 0)
+			(at 100.33 142.24 0)
 			(effects
 				(font
@@
 		)
 		(property "Footprint" "Resistor_SMD:R_1206_3216Metric_Pad1.30x1.75mm_HandSolder"
-			(at 97.028 140.97 90)
+			(at 93.472 140.97 90)
 			(effects
 				(font
@@
 		(dnp no)
 		(property "Reference" "R44"
-			(at 85.09 148.59 0)
+			(at 87.63 146.05 0)
 			(effects
 				(font
@@
 		)
 		(property "Value" "100m"
-			(at 85.09 151.13 0)
-			(effects
-				(font
-					(size 1.27 1.27)
-				)
+			(at 87.63 152.4 0)
+			(effects
+				(font
+					(size 1.27 1.27)
+				)
+				(hide yes)
 			)
 		)
@@
 		(dnp no)
 		(property "Reference" "R45"
-			(at 80.01 156.21 0)
+			(at 82.55 153.67 0)
 			(effects
 				(font
@@
 		)
 		(property "Value" "100m"
-			(at 80.01 158.75 0)
-			(effects
-				(font
-					(size 1.27 1.27)
-				)
-			)
-		)
+			(at 81.28 157.48 0)
+			(effects
+				(font
+					(size 1.27 1.27)
+				)
+				(hide yes)
+			)
+		)
