File: kicad/DC_load/DC_load.kicad_sch (KiCad schematic)
At the start: 4 parts

Commit message: sdf.
Other:
- note removed: "dodaj par LEDova"
Changed lines of the file:
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@@
 		(title "DC load")
-	)
-	(text "dodaj par LEDova\n"
-		(exclude_from_sim no)
-		(at 103.124 79.502 0)
-		(effects
-			(font
-				(size 4 4)
-			)
-		)
 	)
 	(wire
