File: kicad/DC_load/MCU.kicad_sch (KiCad schematic)
At the start: 118 parts, among them J1 BNC, J10 DC fan connector, J6 USB_B, J8 FT232 programming port, J9 Conn_01x04_Socket, Q1 MMBT5401, SW1 RotaryEncoder_Switch, SW2 RotaryEncoder_Switch, SW3 SW_Push, SW8 SW_Push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

Commit message: Schematic done.
Parts:
- removed C42, C43: 47p, Capacitor_SMD:C_0603_1608Metric_Pad1.08x0.95mm_HandSolder, symbol Device:C
- removed C44: 10n, Capacitor_SMD:C_0603_1608Metric_Pad1.08x0.95mm_HandSolder, symbol Device:C
- removed C48: 100n, Capacitor_SMD:C_0603_1608Metric_Pad1.08x0.95mm_HandSolder, symbol Device:C
- removed C57: 10u, Capacitor_SMD:C_0603_1608Metric_Pad1.08x0.95mm_HandSolder, symbol Device:C
- removed J6: USB_B, DC_load:62910416121, symbol Connector:USB_B
- removed R50: 100, Resistor_SMD:R_0603_1608Metric_Pad0.98x0.95mm_HandSolder, symbol Device:R
- removed TP1, TP5: TestPoint, TestPoint:TestPoint_Pad_D2.0mm, symbol Connector:TestPoint
- removed U17: CH340C, Package_SO:SOIC-16_3.9x9.9mm_P1.27mm, symbol DC_load:CH340C
- added J6: Iso board connector, Connector_PinSocket_2.54mm:PinSocket_1x07_P2.54mm_Vertical, symbol Connector:Conn_01x07_Pin
- added Q18: MMBT5401, Package_TO_SOT_SMD:SOT-23, symbol Transistor_BJT:MMBT3906
- added U4: LTV-817S, Package_DIP:SMDIP-4_W9.53mm, symbol Isolator:LTV-817S
- R48, R49: value 22 -> 1k; LCSC C23345 -> C22962
- R64: value 10k -> 1k; LCSC C25804 -> C22962
Connections:
- net 3V3: now also R49.1; no longer R64.1
- net FAN_PWM: no longer J10.4 (Pin_4)
- net GND: now also J6.4 (Pin_4), Q18.3 (C); no longer J10.1 (Pin_1)
- net FAN_PMW_5V: now reaches R48.2
- net FAN_PMW_5V: now also U4.4
- net at R49.2: now also U4.1
- net 5V_EXT: now reaches R48.1
- net 5V_EXT: now also J6.2 (Pin_2)
- net 12V renamed 12V_EXT
- net 12V_EXT: now also J6.3 (Pin_3); no longer TP6.1
- net 5V renamed VCC
- net VCC: now also TP6.1, J6.7 (Pin_7)
- net TACH: no longer names the net of R64.2
- net TACH: now also Q18.1 (B); no longer J10.3 (Pin_3)
- new net: Q18.2 (E), U4.2
- new net Earth: J10.1 (Pin_1), J6.1 (Pin_1), U4.3
- new net FAN_PMW: R64.1
- new net FAN_PWM_5V: J10.4 (Pin_4)
- new net RX_3V3: J6.6 (Pin_6)
- new net TX_3V3: J6.5 (Pin_5)
- no-connect marks 16 -> 10
Other:
- moved on the sheet: C16, C17, C18, C19, C30, C31, C32, C33, C34, C35, C45, C47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

Commit message: Replaced switches with JLCPCB basic.
Parts:
- SW3, SW8: footprint Button_Switch_THT:SW_TH_Tactile_Omron_B3F-10xx -> DC_load:TS-1088-AR02016; LCSC (none) -> C720477
Changed lines of the file:
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@@
 			)
 		)
-		(property "Footprint" "Button_Switch_THT:SW_TH_Tactile_Omron_B3F-10xx"
+		(property "Footprint" "DC_load:TS-1088-AR02016"
 			(at 196.85 43.18 0)
 			(effects
@@
 			)
 		)
+		(property "LCSC" "C720477"
+			(at 201.93 43.18 90)
+			(effects
+				(font
+					(size 1.27 1.27)
+				)
+				(hide yes)
+			)
+		)
 		(pin "2"
 		)
@@
 			)
 		)
-		(property "Footprint" "Button_Switch_THT:SW_TH_Tactile_Omron_B3F-10xx"
+		(property "Footprint" "DC_load:TS-1088-AR02016"
 			(at 167.64 60.96 0)
 			(effects
@@
 			(effects
 				(font
+					(size 1.27 1.27)
+				)
+				(hide yes)
+			)
+		)
+		(property "LCSC" "C720477"
+			(at 172.72 60.96 90)
+			(effects
+				(font

Commit message: Schem Schem.
Parts:
- added J11, J7: Conn_01x02_Pin, Connector_PinHeader_2.54mm:PinHeader_1x02_P2.54mm_Vertical, symbol Connector:Conn_01x02_Pin
- added Q13: MMBT5551L, Package_TO_SOT_SMD:SOT-23, symbol Transistor_BJT:MMBT5551L
- added R50: 10k, Resistor_SMD:R_0603_1608Metric_Pad0.98x0.95mm_HandSolder, symbol Device:R
- added R65: 33k, Resistor_SMD:R_0603_1608Metric_Pad0.98x0.95mm_HandSolder, symbol Device:R
Connections:
- net 12V_EXT: now also R48.1, J11.1 (Pin_1)
- net 5V_EXT: no longer R48.1
- net Earth: now also J7.2 (Pin_2), Q13.2 (E), R50.2
- net FAN_PMW_5V: now also Q13.3 (C), R65.1
- net GND: now also J7.1 (Pin_1)
- net VCC: now also J11.2 (Pin_2)
- new net: Q13.1 (B), R50.1, R65.2
Other:
- note added: "Jumpers when isolation board not used"
- moved on the sheet: J10, J6, Q18, R48, R49, R64, U4

Commit message: M
Parts:
- removed D1, D2: 1N4148W, Diode_SMD:D_SOD-123, symbol Diode:1N4148W
- removed J6: Iso board connector, Connector_PinSocket_2.54mm:PinSocket_1x07_P2.54mm_Vertical, symbol Connector:Conn_01x07_Pin
- added D5: BAV99, Package_TO_SOT_SMD:SOT-23, symbol Diode:BAV99
- added J12: Iso board connector, Connector_PinSocket_2.54mm:PinSocket_1x08_P2.54mm_Vertical, symbol Connector:Conn_01x08_Socket
Connections:
- net 12V_EXT: now also J12.6 (Pin_6)
- net 3V3: now also D5.2 (A), J12.2 (Pin_2)
- net 5V_EXT: now also J12.7 (Pin_7)
- net BNC_CONTROL: now also D5.3 (K)
- net Earth: now also J12.8 (Pin_8)
- net GND: now also D5.1 (K), J12.5 (Pin_5)
- net RX_3V3: now also J12.3 (Pin_3)
- net TX_3V3: now also J12.4 (Pin_4)
- net VCC: now also J12.1 (Pin_1)

Commit message: Connectors fixed.
Parts:
- removed J12: Iso board connector, Connector_PinSocket_2.54mm:PinSocket_1x08_P2.54mm_Vertical, symbol Connector:Conn_01x08_Socket
- removed Q13: MMBT5551L, Package_TO_SOT_SMD:SOT-23, symbol Transistor_BJT:MMBT5551L
- removed R50: 10k, Resistor_SMD:R_0603_1608Metric_Pad0.98x0.95mm_HandSolder, symbol Device:R
- removed R65: 33k, Resistor_SMD:R_0603_1608Metric_Pad0.98x0.95mm_HandSolder, symbol Device:R
- added C42, C43: 100n, Capacitor_SMD:C_0603_1608Metric_Pad1.08x0.95mm_HandSolder, symbol Device:C
- added J13: PC referenced connector, Connector_PinSocket_2.54mm:PinSocket_1x08_P2.54mm_Vertical, symbol Connector:Conn_01x08_Socket
- added J6: Load referenced connector, Connector_PinSocket_2.54mm:PinSocket_1x08_P2.54mm_Vertical, symbol Connector:Conn_01x08_Socket
Connections:
- net 3V3: now also C42.2, J6.7 (Pin_7)
- net Earth: now also C43.1, J13.2 (Pin_2), J13.4 (Pin_4)
- net GND: now also C42.1, J6.2 (Pin_2), J6.4 (Pin_4), J6.6 (Pin_6), J6.8 (Pin_8)
- net RX_3V3: now also J6.3 (Pin_3)
- net TX_3V3: now also J6.5 (Pin_5)
- net VCC: now also J6.1 (Pin_1)
- net 12V_EXT renamed 12V_PC
- net 12V_PC: now also J13.1 (Pin_1); no longer R48.1
- new net 5V_PC: C43.2, R48.1
- new net 5V_PC_PC: J13.3 (Pin_3)
- no-connect marks 10 -> 14
Other:
- moved on the sheet: R49

Commit message: Tiny update.
Parts:
- removed J11: Conn_01x02_Pin, Connector_PinHeader_2.54mm:PinHeader_1x02_P2.54mm_Vertical, symbol Connector:Conn_01x02_Pin
Changed lines of the file:
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@@
 	(wire
 		(pts
-			(xy 232.41 265.43) (xy 234.95 265.43)
-		)
-		(stroke
-			(width 0)
-			(type default)
-		)
-	)
-	(wire
-		(pts
 			(xy 21.59 182.88) (xy 21.59 191.77)
 		)
@@
 	)
 	(symbol
-		(lib_id "power:+5V")
-		(at 234.95 267.97 90)
-		(unit 1)
-		(exclude_from_sim no)
-		(in_bom yes)
-		(on_board yes)
-		(dnp no)
-		(fields_autoplaced yes)
-		(property "Reference" "#PWR0151"
-			(at 238.76 267.97 0)
-			(effects
-				(font
-					(size 1.27 1.27)
-				)
-				(hide yes)
-			)
-		)
-		(property "Value" "VCC"
-			(at 231.14 267.9699 90)
-			(effects
-				(font
-					(size 1.27 1.27)
-				)
-				(justify left)
-			)
-		)
-		(property "Footprint" ""
-			(at 234.95 267.97 0)
-			(effects
-				(font
-					(size 1.27 1.27)
-				)
-				(hide yes)
-			)
-		)
-		(property "Datasheet" ""
-			(at 234.95 267.97 0)
-			(effects
-				(font
-					(size 1.27 1.27)
-				)
-				(hide yes)
-			)
-		)
-		(property "Description" "Power symbol creates a global label with name \"+5V\""
-			(at 234.95 267.97 0)
-			(effects
-				(font
-					(size 1.27 1.27)
-				)
-				(hide yes)
-			)
-		)
-		(pin "1"
-		)
-		(instances
-			(project "DC_load"
-				(path "/ce255642-b081-42cc-af02-07a78c62b42e/57db3589-054f-4b81-a218-89ac743ece5d"
-					(reference "#PWR0151")
-					(unit 1)
-				)
-			)
-		)
-	)
-	(symbol
 		(lib_id "Device:R")
 		(at 72.39 130.81 0)
@@
 	)
 	(symbol
-		(lib_id "Connector:Conn_01x02_Pin")
-		(at 240.03 265.43 0)
-		(mirror y)
-		(unit 1)
-		(exclude_from_sim no)
-		(in_bom yes)
-		(on_board yes)
-		(dnp no)
-		(fields_autoplaced yes)
-		(property "Reference" "J11"
-			(at 241.3 265.4299 0)
-			(effects
-				(font
-					(size 1.27 1.27)
-				)
-				(justify right)
-			)
-		)
-		(property "Value" "Conn_01x02_Pin"
-			(at 241.3 267.9699 0)
-			(effects
-				(font
-					(size 1.27 1.27)
-				)
-				(justify right)
-			)
-		)
-		(property "Footprint" "Connector_PinHeader_2.54mm:PinHeader_1x02_P2.54mm_Vertical"
-			(at 240.03 265.43 0)
-			(effects
-				(font
-					(size 1.27 1.27)
-				)
-				(hide yes)
-			)
-		)
-		(property "Datasheet" "~"
-			(at 240.03 265.43 0)
-			(effects
-				(font
-					(size 1.27 1.27)
-				)
-				(hide yes)
-			)
-		)
-		(property "Description" "Generic connector, single row, 01x02, script generated"
-			(at 240.03 265.43 0)
-			(effects
-				(font
-					(size 1.27 1.27)
-				)
-				(hide yes)
-			)
-		)
-		(pin "2"
-		)
-		(pin "1"
-		)
-		(instances
-			(project "DC_load"
-				(path "/ce255642-b081-42cc-af02-07a78c62b42e/57db3589-054f-4b81-a218-89ac743ece5d"
-					(reference "J11")
-					(unit 1)
-				)
-			)
-		)
-	)
-	(symbol
 		(lib_id "power:GND")
 		(at 347.98 186.69 0)
@@
 					(unit 1)
 				)
-			)
-		)
-	)
-	(symbol
-		(lib_id "power:VCC")
-		(at 232.41 265.43 90)
-		(mirror x)
-		(unit 1)
-		(exclude_from_sim no)
-		(in_bom yes)
-		(on_board yes)
-		(dnp no)
-		(property "Reference" "#PWR0138"
-			(at 236.22 265.43 0)
-			(effects
-				(font
-					(size 1.27 1.27)
-				)
-				(hide yes)
-			)
-		)
-		(property "Value" "12V_PC"
-			(at 229.108 265.43 90)
-			(effects
-				(font
-					(size 1.27 1.27)
-				)
-				(justify left)
-			)
-		)
-		(property "Footprint" ""
-			(at 232.41 265.43 0)
-			(effects
-				(font
-					(size 1.27 1.27)
-				)
-				(hide yes)
-			)
-		)
-		(property "Datasheet" ""
-			(at 232.41 265.43 0)
-			(effects
-				(font
-					(size 1.27 1.27)
-				)
-				(hide yes)
-			)
-		)
-		(property "Description" "Power symbol creates a global label with name \"VCC\""
-			(at 232.41 265.43 0)
-			(effects
-				(font
-					(size 1.27 1.27)
-				)
-				(hide yes)
-			)
-		)
-		(pin "1"
-		)
-		(instances
-			(project "DC_load"
-				(path "/ce255642-b081-42cc-af02-07a78c62b42e/57db3589-054f-4b81-a218-89ac743ece5d"
-					(reference "#PWR0138")
-					(unit 1)
-				)

Commit message: Main board close to done.
Parts:
- added D1, D16: GREEN_LED, LED_SMD:LED_0805_2012Metric_Pad1.15x1.40mm_HandSolder, symbol Device:LED
- added R50, R65: 1k, Resistor_SMD:R_0603_1608Metric_Pad0.98x0.95mm_HandSolder, symbol Device:R
- J13, J6: footprint Connector_PinSocket_2.54mm:PinSocket_1x08_P2.54mm_Vertical -> Connector_PinHeader_2.54mm:PinHeader_1x08_P2.54mm_Vertical
Connections:
- net 5V_PC_PC is gone; now on net 5V_PC: J13.3 (Pin_3)
- net FAN_PMW is gone; now on net FAN_PWM: R64.1
- net FAN_PMW_5V is gone; now on net FAN_PWM_5V: R48.2, U4.4
- net 3V3: now also R50.1
- net GND: now also D1.1 (K), D16.1 (K)
- net at U8.33 (PA12): now also R65.1
- net FAN_BOOST: no longer names the net of U8.32 (PA11)
- new net: D16.2 (A), R50.2
- new net: D1.2 (A), R65.2
- no-connect marks 14 -> 13
Other:
- moved on the sheet: C30, C31, C71, C72, C73, TP3, TP4, U14

Commit message: Fixes
Parts:
- removed R34: 100, Resistor_SMD:R_0603_1608Metric_Pad0.98x0.95mm_HandSolder, symbol Device:R
Changed lines of the file:
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@@
 	)
 	(junction
-		(at 77.47 52.07)
-		(diameter 0)
-		(color 0 0 0 0)
-	)
-	(junction
 		(at 172.72 52.07)
 		(diameter 0)
@@
 	(wire
 		(pts
-			(xy 77.47 52.07) (xy 77.47 59.69)
+			(xy 77.47 48.26) (xy 77.47 59.69)
 		)
 		(stroke
@@
 	(wire
 		(pts
-			(xy 77.47 52.07) (xy 71.12 52.07)
-		)
-		(stroke
-			(width 0)
-			(type default)
-		)
-	)
-	(wire
-		(pts
 			(xy 59.69 199.39) (xy 59.69 201.93)
 		)
@@
 	(wire
 		(pts
-			(xy 58.42 52.07) (xy 63.5 52.07)
-		)
-		(stroke
-			(width 0)
-			(type default)
-		)
-	)
-	(wire
-		(pts
 			(xy 73.66 264.16) (xy 77.47 264.16)
 		)
@@
 	(wire
 		(pts
-			(xy 77.47 48.26) (xy 77.47 52.07)
-		)
-		(stroke
-			(width 0)
-			(type default)
-		)
-	)
-	(wire
-		(pts
 			(xy 142.24 185.42) (xy 142.24 193.04)
 		)
@@
 					(unit 1)
 				)
-			)
-		)
-	)
-	(symbol
-		(lib_id "Device:R")
-		(at 67.31 52.07 270)
-		(mirror x)
-		(unit 1)
-		(exclude_from_sim no)
-		(in_bom yes)
-		(on_board yes)
-		(dnp no)
-		(property "Reference" "R34"
-			(at 62.23 50.292 90)
-			(effects
-				(font
-					(size 1.27 1.27)
-				)
-			)
-		)
-		(property "Value" "100"
-			(at 72.644 50.292 90)
-			(effects
-				(font
-					(size 1.27 1.27)
-				)
-			)
-		)
-		(property "Footprint" "Resistor_SMD:R_0603_1608Metric_Pad0.98x0.95mm_HandSolder"
-			(at 67.31 53.848 90)
-			(effects
-				(font
-					(size 1.27 1.27)
-				)
-				(hide yes)
-			)
-		)
-		(property "Datasheet" "~"
-			(at 67.31 52.07 0)
-			(effects
-				(font
-					(size 1.27 1.27)
-				)
-				(hide yes)
-			)
-		)
-		(property "Description" ""
-			(at 67.31 52.07 0)
-			(effects
-				(font
-					(size 1.27 1.27)
-				)
-			)
-		)
-		(property "LCSC" "C22775"
-			(at 67.31 52.07 0)
-			(effects
-				(font
-					(size 1.27 1.27)
-				)
-				(hide yes)
-			)
-		)
-		(pin "1"
-		)
-		(pin "2"
-		)
-		(instances
-			(project "DC_load"
-				(path "/ce255642-b081-42cc-af02-07a78c62b42e/57db3589-054f-4b81-a218-89ac743ece5d"
-					(reference "R34")
-					(unit 1)
-				)
