File: kicad/DC_load/power_stage.kicad_sch (KiCad schematic)
At the start: 89 parts, among them J2 red_terminal, J3 red terminal, J4 black terminal, J5 black terminal, Q10 MMBT5401, Q11 MMBT5551L, Q12 MMBT5401, Q14 MMBT5551L, Q2 MMBT5401, Q3 FQP19N20C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

Commit message: Ready for production.
Other:
- title: (none) -> Power stage sheet
- moved on the sheet: C74, C75, C8, J2, J5, R10, R14, R15, R19, R29, R30, R32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

Commit message: Schematic done.
Connections:
- net 12V renamed VCC
Changed lines of the file:
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@@
 			)
 		)
-		(property "Value" "12V"
+		(property "Value" "VCC"
 			(at 189.23 124.46 0)
 			(effects
@@
 			)
 		)
-		(property "Value" "12V"
+		(property "Value" "VCC"
 			(at 54.61 31.75 0)
 			(effects
@@
 			)
 		)
-		(property "Value" "12V"
+		(property "Value" "VCC"
 			(at 55.88 124.46 0)
 			(effects
@@
 			)
 		)
-		(property "Value" "12V"
+		(property "Value" "VCC"
 			(at 217.17 124.46 0)
 			(effects
@@
 			)
 		)
-		(property "Value" "12V"
+		(property "Value" "VCC"
 			(at 217.17 31.75 0)
 			(effects
@@
 			)
 		)
-		(property "Value" "12V"
+		(property "Value" "VCC"
 			(at 168.91 124.46 0)
 			(effects
@@
 			)
 		)
-		(property "Value" "12V"
+		(property "Value" "VCC"
 			(at 41.91 31.75 0)
 			(effects
@@
 			)
 		)
-		(property "Value" "12V"
+		(property "Value" "VCC"
 			(at 26.67 124.46 0)
 			(effects
@@
 			)
 		)
-		(property "Value" "12V"
+		(property "Value" "VCC"
 			(at 190.5 31.75 0)
 			(effects
@@
 			)
 		)
-		(property "Value" "12V"
+		(property "Value" "VCC"
 			(at 26.67 31.75 0)
 			(effects
@@
 			)
 		)
-		(property "Value" "12V"
+		(property "Value" "VCC"
 			(at 170.18 31.75 0)
 			(effects
@@
 			)
 		)
-		(property "Value" "12V"
+		(property "Value" "VCC"
 			(at 203.2 31.75 0)
 			(effects
@@
 			)
 		)
-		(property "Value" "12V"
+		(property "Value" "VCC"
 			(at 43.18 124.46 0)
 			(effects
@@
 			)
 		)
-		(property "Value" "12V"
+		(property "Value" "VCC"
 			(at 74.93 31.75 0)
 			(effects
@@
 			)
 		)
-		(property "Value" "12V"
+		(property "Value" "VCC"
 			(at 76.2 124.46 0)
 			(effects
@@
 			)
 		)
-		(property "Value" "12V"
+		(property "Value" "VCC"
 			(at 201.93 124.46 0)
 			(effects

Commit message: Fixes
Changed lines of the file:
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@@
-		)
-	)
-	(polyline
-		(pts
-			(xy 85.09 85.09) (xy 95.25 85.09)
-		)
-		(stroke
-			(width 0)
-			(type default)
 		)
 	)
